File: feedback-jack-board/feedback-jack-board.kicad_sch (KiCad schematic)
At the start: 6 parts, among them J1 Out, J2 Ret, J3 In, J4 Snd, J5 908140508, J6 Barrel_Jack_Switch

Commit message: Jacks board layout
Other:
- company: (none) -> Pedal Markt / Andrei Salomatin
- title: (none) -> RDRPT Jacks Board
Changed lines of the file:
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@@
 (kicad_sch (version 20211123) (generator eeschema)
   (paper "A4")
+  (title_block
+    (title "RDRPT Jacks Board")
+    (date "2025-02-06")
+    (rev "v1rev1")
+    (company "Pedal Markt / Andrei Salomatin")
+  )
   (no_connect (at 30.48 45.72))
   (no_connect (at 81.28 83.82))
