File: feedback-jack-board/feedback-jack-board.kicad_sch (KiCad schematic)
At the start: 6 parts, among them J1 Out, J2 Ret, J3 In, J4 Snd, J5 908140508, J6 Barrel_Jack_Switch

Commit message: jacks board updated
Parts:
- removed J5: 908140508, molex-picoflex8:CONN_SDA-90814_08_MOL, symbol molex-picoflex8:908140508
- added J5: FPC_Connector, Connector_FFC-FPC:JUSHUO_AFA07-S08FCA-00_1x8-1MP_P1.0mm_Horizontal, symbol Connector_Generic_MountingPin:Conn_01x08_MountingPin
Connections:
- net GND: now also J5.4 (Pin_4), J5.7 (Pin_7), J5.MP (MountPin)
- net Gnd: now also J5.1 (Pin_1)
- net In: now also J5.6 (Pin_6)
- net Jack9V: now also J5.8 (Pin_8)
- net Out: now also J5.2 (Pin_2)
- net Ret: now also J5.3 (Pin_3)
- net Snd: now also J5.5 (Pin_5)

Commit message: wip jacks board
Connections:
- net Gnd is gone; now on net GND: J5.1 (Pin_1)
Changed lines of the file:
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@@
+	(wire
+		(pts
+			(xy 133.35 26.67) (xy 138.43 26.67)
+		)
+		(stroke
+			(width 0)
+			(type default)
+		)
+	)
 	(wire
 		(pts
@@
 		)
 	)
-	(label "Gnd"
+	(label "GND"
 		(at 143.51 59.69 180)
 		(effects
@@
 	(label "Out"
 		(at 143.51 62.23 180)
+		(effects
+			(font
+				(size 1.27 1.27)
+			)
+			(justify right bottom)
+		)
+	)
+	(label "GND"
+		(at 133.35 26.67 180)
 		(effects
 			(font
@@
 					(unit 1)
 				)
+			)
+		)
+	)
+	(symbol
+		(lib_id "power:PWR_FLAG")
+		(at 138.43 26.67 0)
+		(unit 1)
+		(body_style 1)
+		(exclude_from_sim no)
+		(in_bom yes)
+		(on_board yes)
+		(in_pos_files yes)
+		(dnp no)
+		(fields_autoplaced yes)
+		(property "Reference" "#FLG01"
+			(at 138.43 24.765 0)
+			(hide yes)
+			(show_name no)
+			(do_not_autoplace no)
+			(effects
+				(font
+					(size 1.27 1.27)
+				)
+			)
+		)
+		(property "Value" "PWR_FLAG"
+			(at 138.43 21.59 0)
+			(show_name no)
+			(do_not_autoplace no)
+			(effects
+				(font
+					(size 1.27 1.27)
+				)
+			)
+		)
+		(property "Footprint" ""
+			(at 138.43 26.67 0)
+			(hide yes)
+			(show_name no)
+			(do_not_autoplace no)
+			(effects
+				(font
+					(size 1.27 1.27)
+				)
+			)
+		)
+		(property "Datasheet" ""
+			(at 138.43 26.67 0)
+			(hide yes)
+			(show_name no)
+			(do_not_autoplace no)
+			(effects
+				(font
+					(size 1.27 1.27)
+				)
+			)
+		)
+		(property "Description" "Special symbol for telling ERC where power comes from"
+			(at 138.43 26.67 0)
+			(hide yes)
+			(show_name no)
+			(do_not_autoplace no)
+			(effects
+				(font
+					(size 1.27 1.27)
+				)
+			)
+		)
+		(pin "1"
+		)
+		(instances
+			(project "feedback-jack-board"
+				(path "/61bcf931-dfc8-433d-a459-074029109891"
+					(reference "#FLG01")
+					(unit 1)
+				)

Commit message: Jacks board v2rev1
Other:
- company: Pedal Markt / Andrei Salomatin -> Andrei Salomatin / akkusativ
Changed lines of the file:
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@@
 	(title_block
 		(title "RDRPT Jacks Board")
-		(date "2025-02-06")
-		(rev "v1rev1")
-		(company "Pedal Markt / Andrei Salomatin")
+		(date "2026-10-18")
+		(rev "v2rev1")
+		(company "Andrei Salomatin / akkusativ")
 	)
 	(no_connect
