File: feedback-jack-board/feedback-jack-board.kicad_pcb (KiCad board)
At the start: 2 copper layers, 77.5 x 37 mm, 12 parts, among them J1 Out, J2 Ret, J3 In, J4 Snd, J5 FPC_Connector, J6 Barrel_Jack_Switch

Commit message: wip jacks board
Connections:
- J5 pad 1: /Gnd -> GND
Changed lines of the file:
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@@
 		(sheetname "/")
 		(sheetfile "feedback-jack-board.kicad_sch")
-		(units
-			(unit
-				(name "A")
-				(pins "S" "R" "RN" "T" "TN")
-			)
-		)
 		(attr through_hole)
 		(duplicate_pad_numbers_are_jumpers no)
@@
 		)
 		(fp_line
-			(start 8 -9.8)
-			(end 8 7)
+			(start 8 -9.4)
+			(end 8 6.6)
 			(stroke
 				(width 0.05)
@@
 		)
 		(fp_line
-			(start -26.5 -9.8)
-			(end 8 -9.8)
+			(start -26.5 -9.4)
+			(end 8 -9.4)
 			(stroke
 				(width 0.05)
@@
 		)
 		(fp_line
-			(start 8 7)
-			(end -26.5 7)
+			(start 8 6.6)
+			(end -26.5 6.6)
 			(stroke
 				(width 0.05)
@@
 		)
 		(fp_line
-			(start -26.5 7)
-			(end -26.5 -9.8)
+			(start -26.5 6.6)
+			(end -26.5 -9.4)
 			(stroke
 				(width 0.05)
@@
 		(sheetname "/")
 		(sheetfile "feedback-jack-board.kicad_sch")
-		(units
-			(unit
-				(name "A")
-				(pins "S" "R" "RN" "T" "TN")
-			)
-		)
 		(attr through_hole)
 		(duplicate_pad_numbers_are_jumpers no)
@@
 		)
 		(fp_line
-			(start 8 -9.8)
-			(end 8 7)
+			(start 8 -9.4)
+			(end 8 6.6)
 			(stroke
 				(width 0.05)
@@
 		)
 		(fp_line
-			(start -26.5 -9.8)
-			(end 8 -9.8)
+			(start -26.5 -9.4)
+			(end 8 -9.4)
 			(stroke
 				(width 0.05)
@@
 		)
 		(fp_line
-			(start 8 7)
-			(end -26.5 7)
+			(start 8 6.6)
+			(end -26.5 6.6)
 			(stroke
 				(width 0.05)
@@
 		)
 		(fp_line
-			(start -26.5 7)
-			(end -26.5 -9.8)
+			(start -26.5 6.6)
+			(end -26.5 -9.4)
 			(stroke
 				(width 0.05)
@@
 		(sheetname "/")
 		(sheetfile "feedback-jack-board.kicad_sch")
-		(units
-			(unit
-				(name "A")
-				(pins "S" "R" "RN" "T" "TN")
-			)
-		)
 		(attr through_hole)
 		(duplicate_pad_numbers_are_jumpers no)
@@
 		)
 		(fp_line
-			(start 8 -9.8)
-			(end 8 7)
+			(start 8 -9.4)
+			(end 8 6.6)
 			(stroke
 				(width 0.05)
@@
 		)
 		(fp_line
-			(start -26.5 -9.8)
-			(end 8 -9.8)
+			(start -26.5 -9.4)
+			(end 8 -9.4)
 			(stroke
 				(width 0.05)
@@
 		)
 		(fp_line
-			(start 8 7)
-			(end -26.5 7)
+			(start 8 6.6)
+			(end -26.5 6.6)
 			(stroke
 				(width 0.05)
@@
 		)
 		(fp_line
-			(start -26.5 7)
-			(end -26.5 -9.8)
+			(start -26.5 6.6)
+			(end -26.5 -9.4)
 			(stroke
 				(width 0.05)
@@
 		(sheetname "/")
 		(sheetfile "feedback-jack-board.kicad_sch")
-		(units
-			(unit
-				(name "A")
-				(pins "S" "R" "RN" "T" "TN")
-			)
-		)
 		(attr through_hole)
 		(duplicate_pad_numbers_are_jumpers no)
@@
 		)
 		(fp_line
-			(start 8 -9.8)
-			(end 8 7)
+			(start 8 -9.4)
+			(end 8 6.6)
 			(stroke
 				(width 0.05)
@@
 		)
 		(fp_line
-			(start -26.5 -9.8)
-			(end 8 -9.8)
+			(start -26.5 -9.4)
+			(end 8 -9.4)
 			(stroke
 				(width 0.05)
@@
 		)
 		(fp_line
-			(start 8 7)
-			(end -26.5 7)
+			(start 8 6.6)
+			(end -26.5 6.6)
 			(stroke
 				(width 0.05)
@@
 		)
 		(fp_line
-			(start -26.5 7)
-			(end -26.5 -9.8)
+			(start -26.5 6.6)
+			(end -26.5 -9.4)
 			(stroke
 				(width 0.05)
@@
 			(layers "F.Cu" "F.Mask" "F.Paste")
 			(roundrect_rratio 0.25)
-			(net "/Gnd")
+			(net "GND")
 			(pinfunction "Pin_1_1")
 			(pintype "passive")
