File: feedback-main-board/core.kicad_sch (KiCad schematic)
At the start: 43 parts

Commit message: Board started
Parts:
- removed C? (x4): 100n, symbol Device:C
- removed D? (x2): LED, symbol Device:LED
- removed R?: 100k, symbol Device:R
- added C14: 100n, Capacitor_SMD:C_0603_1608Metric_Pad1.08x0.95mm_HandSolder, symbol Device:C
- added C8: 2u2, Capacitor_THT:C_Rect_L7.2mm_W7.2mm_P5.00mm_FKS2_FKP2_MKS2_MKP2, symbol Device:C
- added R10: 100, Resistor_SMD:R_0603_1608Metric_Pad0.98x0.95mm_HandSolder, symbol Device:R
- added R12: 10k, Resistor_SMD:R_0603_1608Metric_Pad0.98x0.95mm_HandSolder, symbol Device:R
- added R8: 100k, Resistor_SMD:R_0603_1608Metric_Pad0.98x0.95mm_HandSolder, symbol Device:R
- added unit 5 of U1
- added unit 1 of U2
- C10, C11, C15, C5: renamed from C?; footprint (none) -> Capacitor_SMD:C_0603_1608Metric_Pad1.08x0.95mm_HandSolder
- C12, C7: renamed from C?; footprint (none) -> Capacitor_THT:C_Rect_L7.2mm_W7.2mm_P5.00mm_FKS2_FKP2_MKS2_MKP2
- C13, C9: renamed from C?; value 1u -> 2u2; footprint (none) -> Capacitor_THT:C_Rect_L7.2mm_W7.2mm_P5.00mm_FKS2_FKP2_MKS2_MKP2
- C6: renamed from C?; footprint (none) -> Capacitor_THT:C_Rect_L7.0mm_W4.5mm_P5.00mm
- D2, D3, D4, D5: renamed from D?; footprint (none) -> Diode_THT:D_A-405_P7.62mm_Horizontal
- R11, R13, R14, R15, R16, R17, R19, R5, R6, R7, R9: renamed from R?; footprint (none) -> Resistor_SMD:R_0603_1608Metric_Pad0.98x0.95mm_HandSolder
- R18: renamed from R?; value 1k -> 100; footprint (none) -> Resistor_SMD:R_0603_1608Metric_Pad0.98x0.95mm_HandSolder
- R20: renamed from R?; footprint (none) -> Resistor_SMD:R_0603_1608Metric_Pad0.98x0.95mm_HandSolder; Mouser 603-RT0603DRE07100KL -> (none)
- RV1, RV2, RV3: renamed from RV?; value A100k -> A10k
- SW1, SW2: renamed from SW?; footprint (none) -> MBP switches:SPDT.LUGS.PM
- U1, U2: renamed from U?; footprint (none) -> Package_SO:SOIC-14_3.9x8.7mm_P1.27mm
Connections:
- net +4V5: now also RV2.1, U2.12 (+), R12.1, R8.2; no longer U2.5 (+)
- net +9V: now also C14.2, U1.4 (V+)
- net Feedback: now also SW2.3 (C); no longer SW2.2 (B)
- net GND: now also C14.1, U1.11 (V-); no longer RV2.1
- net at SW1.2 (B): now also U2.5 (+); no longer U2.10 (+)
- net at C11.2, R17.2, R19.1: now also U2.7; no longer U2.8
- net at C11.1, R15.2, R17.1: now also U2.6 (-); no longer U2.9 (-)
- net OutPreVol: now reaches C9.2, RV2.3
- net OutPreVol: now also SW2.1 (A)
- net at D2.1 (K), D4.2 (A): now also SW2.2 (B); no longer SW2.1 (A)
- net at C10.2, R16.2, R18.1: now also U2.14; no longer U2.7
- net at C10.1, R13.2, R14.2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: now also U2.13 (-); no longer U2.6 (-)
- net Out renamed FxOut
- net ToInvert renamed RetBuf
- net RetBuf: now also U2.10 (+), C8.2, R12.2; no longer C6.2, U2.12 (+)
- new net: C6.2, R8.1, U2.3 (+)
- new net: C8.1, R10.2
- new net: R10.1, U2.1, U2.2 (-)
- new net: R11.1, U2.8, U2.9 (-)
Other:
- note added: "On-Off-On"
- note added: "Try 2u2/A10K in case of clicks everywhere pre-DG403"
- moved on the sheet: C10, C12, C15, C6, C9, D2, D3, D4, D5, R11, R13, R14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

Commit message: Component placement
Connections:
- net +4V5: now also U2.10 (+); no longer U2.12 (+)
- net RetBuf: now also U2.12 (+); no longer U2.10 (+)
- net at SW1.2 (B): now also U2.3 (+); no longer U2.5 (+)
- net at C11.1, R15.2, R17.1: now also U2.2 (-); no longer U2.6 (-)
- net at C11.2, R17.2, R19.1: now also U2.1; no longer U2.7
- net at C6.2, R8.1: now also U2.5 (+); no longer U2.3 (+)
- net at C5.2, R7.1: now also U1.10 (+); no longer U1.3 (+)
- net at C10.2, R16.2, R18.1: now also U2.8; no longer U2.14
- net at C10.1, R13.2, R14.2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: now also U2.9 (-); no longer U2.13 (-)
- new net: R9.1, U1.8, U1.9 (-)
- new net: R10.1, U2.6 (-), U2.7
- new net: R11.1, U2.13 (-), U2.14
Changed lines of the file:
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@@
     (effects (font (size 1.27 1.27)) (justify right))
   )
-  (symbol (lib_id "Amplifier_Operational:TL074") (at 167.64 48.26 0) (mirror x) (unit 2)
+  (symbol (lib_id "Amplifier_Operational:TL074") (at 167.64 48.26 0) (mirror x) (unit 1)
     (in_bom yes) (on_board yes) (fields_autoplaced)
     (property "Reference" "U2" (id 0) (at 167.64 38.1 0))
@@
     (pin "2")
   )
-  (symbol (lib_id "Amplifier_Operational:TL074") (at 57.15 171.45 0) (mirror x) (unit 3)
+  (symbol (lib_id "Amplifier_Operational:TL074") (at 57.15 171.45 0) (mirror x) (unit 4)
     (in_bom yes) (on_board yes) (fields_autoplaced)
     (property "Reference" "U2" (id 0) (at 57.15 161.29 0))
@@
     (pin "2")
   )
-  (symbol (lib_id "Amplifier_Operational:TL074") (at 57.15 114.3 0) (mirror x) (unit 1)
+  (symbol (lib_id "Amplifier_Operational:TL074") (at 57.15 114.3 0) (mirror x) (unit 2)
     (in_bom yes) (on_board yes) (fields_autoplaced)
     (property "Reference" "U2" (id 0) (at 57.15 104.14 0))
@@
     (pin "2")
   )
-  (symbol (lib_id "Amplifier_Operational:TL074") (at 58.42 48.26 0) (mirror x) (unit 1)
+  (symbol (lib_id "Amplifier_Operational:TL074") (at 58.42 48.26 0) (mirror x) (unit 3)
     (in_bom yes) (on_board yes) (fields_autoplaced)
     (property "Reference" "U1" (id 0) (at 58.42 38.1 0))
@@
     (pin "2")
   )
-  (symbol (lib_id "Amplifier_Operational:TL074") (at 166.37 114.3 0) (mirror x) (unit 4)
+  (symbol (lib_id "Amplifier_Operational:TL074") (at 166.37 114.3 0) (mirror x) (unit 3)
     (in_bom yes) (on_board yes) (fields_autoplaced)
     (property "Reference" "U2" (id 0) (at 166.37 104.14 0))

Commit message: Routing v1 done
Parts:
- C5: footprint Capacitor_SMD:C_0603_1608Metric_Pad1.08x0.95mm_HandSolder -> Capacitor_THT:C_Rect_L7.0mm_W2.5mm_P5.00mm
Changed lines of the file:
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@@
     (property "Reference" "C5" (id 0) (at 35.56 43.18 90))
     (property "Value" "100n" (id 1) (at 35.56 45.72 90))
-    (property "Footprint" "Capacitor_SMD:C_0603_1608Metric_Pad1.08x0.95mm_HandSolder" (id 2) (at 39.37 49.8348 0)
+    (property "Footprint" "Capacitor_THT:C_Rect_L7.0mm_W2.5mm_P5.00mm" (id 2) (at 39.37 49.8348 0)
       (effects (font (size 1.27 1.27)) hide)
     )

Commit message: Mouser parts ordered
Parts:
- C12, C13, C7, C8, C9: Mouser (none) -> 505-MKS22.2/63/5
- C6: Mouser (none) -> 505-MKS2-1/63/10A
- U1, U2: Mouser (none) -> 595-TL074IDR
Changed lines of the file:
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@@
+      (effects (font (size 1.27 1.27)) hide)
+    )
+    (property "Mouser" "595-TL074IDR" (id 4) (at 167.64 48.26 0)
       (effects (font (size 1.27 1.27)) hide)
     )
@@
       (effects (font (size 1.27 1.27)) hide)
     )
+    (property "Mouser" "505-MKS2-1/63/10A" (id 4) (at 35.56 116.84 0)
+      (effects (font (size 1.27 1.27)) hide)
+    )
     (pin "1")
     (pin "2")
@@
       (effects (font (size 1.27 1.27)) hide)
     )
+    (property "Mouser" "505-MKS22.2/63/5" (id 4) (at 85.09 171.45 0)
+      (effects (font (size 1.27 1.27)) hide)
+    )
     (pin "1")
     (pin "2")
@@
       (effects (font (size 1.27 1.27)) hide)
     )
+    (property "Mouser" "505-MKS22.2/63/5" (id 4) (at 85.09 114.3 0)
+      (effects (font (size 1.27 1.27)) hide)
+    )
     (pin "1")
     (pin "2")
@@
     )
     (property "Datasheet" "http://www.ti.com/lit/ds/symlink/tl071.pdf" (id 3) (at 279.4 30.48 0)
+      (effects (font (size 1.27 1.27)) hide)
+    )
+    (property "Mouser" "595-TL074IDR" (id 4) (at 278.13 35.56 0)
       (effects (font (size 1.27 1.27)) hide)
     )
@@
       (effects (font (size 1.27 1.27)) hide)
     )
+    (property "Mouser" "505-MKS22.2/63/5" (id 4) (at 194.31 114.3 0)
+      (effects (font (size 1.27 1.27)) hide)
+    )
     (pin "1")
     (pin "2")
@@
       (effects (font (size 1.27 1.27)) hide)
     )
+    (property "Mouser" "505-MKS22.2/63/5" (id 4) (at 85.09 48.26 0)
+      (effects (font (size 1.27 1.27)) hide)
+    )
     (pin "1")
     (pin "2")
@@
     )
     (property "Datasheet" "http://www.ti.com/lit/ds/symlink/tl071.pdf" (id 3) (at 257.175 30.48 0)
+      (effects (font (size 1.27 1.27)) hide)
+    )
+    (property "Mouser" "595-TL074IDR" (id 4) (at 255.905 35.56 0)
       (effects (font (size 1.27 1.27)) hide)
     )
@@
       (effects (font (size 1.27 1.27)) hide)
     )
+    (property "Mouser" "595-TL074IDR" (id 4) (at 57.15 171.45 0)
+      (effects (font (size 1.27 1.27)) hide)
+    )
     (pin "1")
     (pin "2")
@@
       (effects (font (size 1.27 1.27)) hide)
     )
+    (property "Mouser" "595-TL074IDR" (id 4) (at 57.15 114.3 0)
+      (effects (font (size 1.27 1.27)) hide)
+    )
     (pin "1")
     (pin "2")
@@
       (effects (font (size 1.27 1.27)) hide)
     )
+    (property "Mouser" "595-TL074IDR" (id 4) (at 58.42 48.26 0)
+      (effects (font (size 1.27 1.27)) hide)
+    )
     (pin "1")
     (pin "2")
@@
       (effects (font (size 1.27 1.27)) hide)
     )
+    (property "Mouser" "595-TL074IDR" (id 4) (at 166.37 114.3 0)
+      (effects (font (size 1.27 1.27)) hide)
+    )
     (pin "1")
     (pin "2")
@@
       (effects (font (size 1.27 1.27)) hide)
     )
+    (property "Mouser" "505-MKS22.2/63/5" (id 4) (at 198.12 48.26 0)
+      (effects (font (size 1.27 1.27)) hide)
+    )

Commit message: Wip rev2
Connections:
- net +4V5: now also SW1.3 (C); no longer SW1.1 (A)
- net RetBuf: now also SW1.1 (A); no longer SW1.3 (C)
Other:
- moved on the sheet: SW1
Changed lines of the file:
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@@
     (pin "4")
   )
-  (symbol (lib_id "Switch:SW_SPDT") (at 152.4 57.15 0) (mirror y) (unit 1)
+  (symbol (lib_id "Switch:SW_SPDT") (at 152.4 57.15 180) (unit 1)
     (in_bom yes) (on_board yes) (fields_autoplaced)
     (property "Reference" "SW1" (id 0) (at 152.4 49.53 0))
