File: feedback-main-board/core.kicad_sch (KiCad schematic)
At the start: 38 parts, among them SW1 SW_SPDT, SW2 SW_SPDT, U1 TL074, U2 TL074

Commit message: JLCPCB rev3 ordered
Parts:
- U1, U2: value TL074 -> OPA1679; LCSC C6964 -> C2878631; Mouser 595-TL074IDR -> (none)
Changed lines of the file:
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@@
     (in_bom yes) (on_board yes) (fields_autoplaced)
     (property "Reference" "U2" (id 0) (at 167.64 38.1 0))
-    (property "Value" "TL074" (id 1) (at 167.64 40.64 0))
+    (property "Value" "OPA1679" (id 1) (at 167.64 40.64 0))
     (property "Footprint" "Package_SO:SOIC-14_3.9x8.7mm_P1.27mm" (id 2) (at 166.37 50.8 0)
       (effects (font (size 1.27 1.27)) hide)
@@
       (effects (font (size 1.27 1.27)) hide)
     )
-    (property "Mouser" "595-TL074IDR" (id 4) (at 167.64 48.26 0)
-      (effects (font (size 1.27 1.27)) hide)
-    )
-    (property "LCSC" "C6964" (id 5) (at 167.64 48.26 0)
+    (property "Mouser" "" (id 4) (at 167.64 48.26 0)
+      (effects (font (size 1.27 1.27)) hide)
+    )
+    (property "LCSC" "C2878631" (id 5) (at 167.64 48.26 0)
       (effects (font (size 1.27 1.27)) hide)
     )
@@
       (effects (font (size 1.27 1.27)) (justify left))
     )
-    (property "Value" "TL074" (id 1) (at 276.86 36.8299 0)
+    (property "Value" "OPA1679" (id 1) (at 276.86 36.8299 0)
       (effects (font (size 1.27 1.27)) (justify left))
     )
@@
       (effects (font (size 1.27 1.27)) hide)
     )
-    (property "Mouser" "595-TL074IDR" (id 4) (at 278.13 35.56 0)
-      (effects (font (size 1.27 1.27)) hide)
-    )
-    (property "LCSC" "C6964" (id 5) (at 278.13 35.56 0)
+    (property "Mouser" "" (id 4) (at 278.13 35.56 0)
+      (effects (font (size 1.27 1.27)) hide)
+    )
+    (property "LCSC" "C2878631" (id 5) (at 278.13 35.56 0)
       (effects (font (size 1.27 1.27)) hide)
     )
@@
       (effects (font (size 1.27 1.27)) (justify left))
     )
-    (property "Value" "TL074" (id 1) (at 254.635 36.8299 0)
+    (property "Value" "OPA1679" (id 1) (at 254.635 36.8299 0)
       (effects (font (size 1.27 1.27)) (justify left))
     )
@@
       (effects (font (size 1.27 1.27)) hide)
     )
-    (property "Mouser" "595-TL074IDR" (id 4) (at 255.905 35.56 0)
-      (effects (font (size 1.27 1.27)) hide)
-    )
-    (property "LCSC" "C6964" (id 5) (at 255.905 35.56 0)
+    (property "Mouser" "" (id 4) (at 255.905 35.56 0)
+      (effects (font (size 1.27 1.27)) hide)
+    )
+    (property "LCSC" "C2878631" (id 5) (at 255.905 35.56 0)
       (effects (font (size 1.27 1.27)) hide)
     )
@@
     (in_bom yes) (on_board yes) (fields_autoplaced)
     (property "Reference" "U2" (id 0) (at 57.15 161.29 0))
-    (property "Value" "TL074" (id 1) (at 57.15 163.83 0))
+    (property "Value" "OPA1679" (id 1) (at 57.15 163.83 0))
     (property "Footprint" "Package_SO:SOIC-14_3.9x8.7mm_P1.27mm" (id 2) (at 55.88 173.99 0)
       (effects (font (size 1.27 1.27)) hide)
@@
       (effects (font (size 1.27 1.27)) hide)
     )
-    (property "Mouser" "595-TL074IDR" (id 4) (at 57.15 171.45 0)
-      (effects (font (size 1.27 1.27)) hide)
-    )
-    (property "LCSC" "C6964" (id 5) (at 57.15 171.45 0)
+    (property "Mouser" "" (id 4) (at 57.15 171.45 0)
+      (effects (font (size 1.27 1.27)) hide)
+    )
+    (property "LCSC" "C2878631" (id 5) (at 57.15 171.45 0)
       (effects (font (size 1.27 1.27)) hide)
     )
@@
     (in_bom yes) (on_board yes) (fields_autoplaced)
     (property "Reference" "U2" (id 0) (at 57.15 104.14 0))
-    (property "Value" "TL074" (id 1) (at 57.15 106.68 0))
+    (property "Value" "OPA1679" (id 1) (at 57.15 106.68 0))
     (property "Footprint" "Package_SO:SOIC-14_3.9x8.7mm_P1.27mm" (id 2) (at 55.88 116.84 0)
       (effects (font (size 1.27 1.27)) hide)
@@
       (effects (font (size 1.27 1.27)) hide)
     )
-    (property "Mouser" "595-TL074IDR" (id 4) (at 57.15 114.3 0)
-      (effects (font (size 1.27 1.27)) hide)
-    )
-    (property "LCSC" "C6964" (id 5) (at 57.15 114.3 0)
+    (property "Mouser" "" (id 4) (at 57.15 114.3 0)
+      (effects (font (size 1.27 1.27)) hide)
+    )
+    (property "LCSC" "C2878631" (id 5) (at 57.15 114.3 0)
       (effects (font (size 1.27 1.27)) hide)
     )
@@
     (in_bom yes) (on_board yes) (fields_autoplaced)
     (property "Reference" "U1" (id 0) (at 58.42 38.1 0))
-    (property "Value" "TL074" (id 1) (at 58.42 40.64 0))
+    (property "Value" "OPA1679" (id 1) (at 58.42 40.64 0))
     (property "Footprint" "Package_SO:SOIC-14_3.9x8.7mm_P1.27mm" (id 2) (at 57.15 50.8 0)
       (effects (font (size 1.27 1.27)) hide)
@@
       (effects (font (size 1.27 1.27)) hide)
     )
-    (property "Mouser" "595-TL074IDR" (id 4) (at 58.42 48.26 0)
-      (effects (font (size 1.27 1.27)) hide)
-    )
-    (property "LCSC" "C6964" (id 5) (at 58.42 48.26 0)
+    (property "Mouser" "" (id 4) (at 58.42 48.26 0)
+      (effects (font (size 1.27 1.27)) hide)
+    )
+    (property "LCSC" "C2878631" (id 5) (at 58.42 48.26 0)
       (effects (font (size 1.27 1.27)) hide)
     )
@@
     (in_bom yes) (on_board yes) (fields_autoplaced)
     (property "Reference" "U2" (id 0) (at 166.37 104.14 0))
-    (property "Value" "TL074" (id 1) (at 166.37 106.68 0))
+    (property "Value" "OPA1679" (id 1) (at 166.37 106.68 0))
     (property "Footprint" "Package_SO:SOIC-14_3.9x8.7mm_P1.27mm" (id 2) (at 165.1 116.84 0)
       (effects (font (size 1.27 1.27)) hide)
@@
       (effects (font (size 1.27 1.27)) hide)
     )
-    (property "Mouser" "595-TL074IDR" (id 4) (at 166.37 114.3 0)
-      (effects (font (size 1.27 1.27)) hide)
-    )
-    (property "LCSC" "C6964" (id 5) (at 166.37 114.3 0)
-      (effects (font (size 1.27 1.27)) hide)
-    )
+    (property "Mouser" "" (id 4) (at 166.37 114.3 0)
+      (effects (font (size 1.27 1.27)) hide)
+    )
+    (property "LCSC" "C2878631" (id 5) (at 166.37 114.3 0)
+      (effects (font (size 1.27 1.27)) hide)
+    )
