File: feedback-main-board/core.kicad_sch (KiCad schematic)
At the start: 38 parts, among them SW1 SW_SPDT, SW2 SW_SPDT, U1 OPA1679, U2 OPA1679

Commit message: wip
Parts:
- removed C12, C13, C7, C8, C9: 2u2, Capacitor_THT:C_Rect_L7.2mm_W7.2mm_P5.00mm_FKS2_FKP2_MKS2_MKP2, symbol Device:C
- added C? (x9): 47u, Capacitor_SMD:CP_Elec_5x5.4, symbol Device:C_Polarized
- added R? (x2): 10k, Resistor_SMD:R_0603_1608Metric_Pad0.98x0.95mm_HandSolder, symbol Device:R
- C6: value 1u -> 100n; footprint Capacitor_THT:C_Rect_L7.0mm_W4.5mm_P5.00mm -> Capacitor_THT:C_Rect_L7.0mm_W2.5mm_P5.00mm; Mouser 505-MKS2-1/63/10A -> (none)
- D2, D3, D4, D5: value D -> 1N4148; footprint Diode_THT:D_A-405_P7.62mm_Horizontal -> Diode_SMD:D_SOD-323; LCSC DNP -> C2128
- R6, R8: value 100k -> 1M; LCSC C25803 -> C22935
- RV1, RV2, RV3: value A10k -> A500k
Connections:
- net +4V5: now also R?.1, R?.1; no longer D3.2 (A), D5.1 (K), RV1.1, RV2.1, RV3.1
- net Feedback: now also C?.2; no longer R14.1
- net FxOut: now also C?.1, R?.2; no longer RV2.2
- net InBuf: now also C?.1, R?.2; no longer RV1.3
- net InGain: now also C?.2; no longer R13.1
- net OutPreVol: now also C?.2
- net PreFeedback: now also C?.2
- net RetBuf: now also C?.2
- net Sum: now also C?.2
- net at R9.2: now also C?.1
- net at R11.2: now also C?.1
- net at R10.2: now also C?.1
- net at R19.2: now also C?.1
- net at R18.2: now also C?.1
- net GND renamed SIG_GND
- net SIG_GND: now also D3.2 (A), D5.1 (K), RV1.1, RV2.1, RV3.1; no longer C14.1, C15.1, U1.11 (V-), U2.11 (V-)
- new net: C?.2, C?.2, RV1.3
- new net: C?.2, RV2.2
- new net: C?.1, R13.1
- new net: C?.1, R14.1
- new net PWR_GND: C14.1, C15.1, U1.11 (V-), U2.11 (V-)
Other:
- note removed: "Try 2u2/A10K in case of clicks everywhere pre-DG403"
- moved on the sheet: D4, D5, RV2

Commit message: wip
Parts:
- added C7, C8: 220p, Capacitor_SMD:C_0603_1608Metric_Pad1.08x0.95mm_HandSolder, symbol Device:C
- added R46, R47: 4.7k, Resistor_SMD:R_0603_1608Metric_Pad0.98x0.95mm_HandSolder, symbol Device:R
- C5, C6: footprint Capacitor_THT:C_Rect_L7.0mm_W2.5mm_P5.00mm -> Capacitor_SMD:C_1206_3216Metric_Pad1.33x1.80mm_HandSolder; LCSC DNP -> C97946
- D2, D3, D4, D5: footprint Diode_SMD:D_SOD-323 -> Diode_SMD:D_SOD-323_HandSoldering
- gave numbers to parts that had none: 11
Connections:
- net SIG_GND is gone; now on net GND: D3.2 (A), D5.1 (K), R5.2, R6.2, RV1.0 (ShieldPin), RV1.1, RV2.0 (ShieldPin), RV2.1, RV3.0 (ShieldPin), RV3.1
- net at C6.2, R8.1: now also R47.1; no longer U2.5 (+)
- net at C5.2, R7.1: now also R46.1; no longer U1.10 (+)
- net PWR_GND renamed GND
- net GND: now also C7.2, C8.2
- new net: C8.1, R47.2, U2.5 (+)
- new net: C7.1, R46.2, U1.10 (+)
Other:
- moved on the sheet: C5, C6, R5, R6, R7, R8

Commit message: wip jacks board
Other:
- company: Pedal Markt / Andrei Salomatin -> Andrei Salomatin / akkusativ
- title: Read/Repeat -> RDRPT
- moved on the sheet: D2, D3, SW2, U1E
