File: feedback-main-board/feedback-main-board.kicad_sch (KiCad schematic)
At the start: 9 parts

Commit message: Board started
Parts:
- removed C? (x2): 10u, symbol Device:C_Polarized
- removed C?: 1u, symbol Device:C_Polarized
- removed R? (x2): 10k, symbol Device:R
- added C2: 10u, Capacitor_SMD:CP_Elec_5x5.4, symbol Device:C_Polarized
- added C3: 10u, Capacitor_SMD:CP_Elec_4x5.4, symbol Device:C_Polarized
- added C4: 100n, Capacitor_SMD:C_0603_1608Metric_Pad1.08x0.95mm_HandSolder, symbol Device:C
- added J1: 908140508, molex-picoflex8:CONN_SDA-90814_08_MOL, symbol molex-picoflex8:908140508
- added J2: FLIP, Connector_JST:JST_XH_B2B-XH-A_1x02_P2.50mm_Vertical, symbol Connector:Conn_01x02_Male
- added J3: RPT, Connector_JST:JST_XH_B2B-XH-A_1x02_P2.50mm_Vertical, symbol Connector:Conn_01x02_Male
- added R2, R3: 10K, Resistor_SMD:R_0603_1608Metric_Pad0.98x0.95mm_HandSolder, symbol Device:R
- added R4: 10, Resistor_SMD:R_0603_1608Metric_Pad0.98x0.95mm_HandSolder, symbol Device:R
- added U1: TL074, Package_SO:SOIC-14_3.9x8.7mm_P1.27mm, symbol Amplifier_Operational:TL074
- C1: renamed from C?; footprint (none) -> Capacitor_SMD:CP_Elec_6.3x5.4; LCSC (none) -> C4747963
- gave numbers to parts that had none: 3
Connections:
- net +4V5: now also C3.1, C4.2, R4.2
- net +9V: now also J2.2 (Pin_2), R2.1
- net GND: now also C2.2, C3.2, C4.1, J1.2, J1.5, J1.8, R3.2
- net Jack9V: now also J1.1
- new net: C2.1, R2.2, R3.1, U1.10 (+)
- new net: R4.1, U1.8, U1.9 (-)
- new net In: J1.3
- new net LatchSw1: J3.1 (Pin_1)
- new net LatchSw2: J3.2 (Pin_2)
- new net MomSw1: J2.1 (Pin_1)
- new net Out: J1.7
- new net Ret: J1.6
- new net Snd: J1.4
Other:
- sheet Core ports: added FxOut, RetBuf; removed Out
- sheet Switching ports: added FxOut, LatchSw1, LatchSw2, MomSwIn, Out, RetBuf; removed none

Commit message: Component placement
Parts:
- C3: footprint Capacitor_SMD:CP_Elec_4x5.4 -> Capacitor_SMD:CP_Elec_5x5.4
Connections:
- net at C2.1, R2.2, R3.1: now also U1.12 (+); no longer U1.10 (+)
- new net: R4.1, U1.13 (-), U1.14
Changed lines of the file:
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@@
     (pin "2")
   )
-  (symbol (lib_id "Amplifier_Operational:TL074") (at 119.38 175.26 0) (mirror x) (unit 3)
+  (symbol (lib_id "Amplifier_Operational:TL074") (at 119.38 175.26 0) (mirror x) (unit 4)
     (in_bom yes) (on_board yes) (fields_autoplaced)
     (property "Reference" "U1" (id 0) (at 119.38 165.1 0))
@@
       (effects (font (size 1.27 1.27)) (justify right))
     )
-    (property "Footprint" "Capacitor_SMD:CP_Elec_4x5.4" (id 2) (at 144.4752 185.42 0)
+    (property "Footprint" "Capacitor_SMD:CP_Elec_5x5.4" (id 2) (at 144.4752 185.42 0)
       (effects (font (size 1.27 1.27)) hide)
     )
@@
     )
     (path "/6f26c93d-3421-4b4c-a96f-4f7610302b66"
-      (reference "C3") (unit 1) (value "10u") (footprint "Capacitor_SMD:CP_Elec_4x5.4")
+      (reference "C3") (unit 1) (value "10u") (footprint "Capacitor_SMD:CP_Elec_5x5.4")
     )
     (path "/e9573214-ca11-4174-9555-8f03d24e4d9c"
@@
       (reference "SW2") (unit 1) (value "SW_SPDT") (footprint "MBP switches:SPDT.LUGS.PM")
     )
-    (path "/1c9013f3-dc47-4074-b623-b743c64985e1/e0a84abb-9577-4377-ad97-14afdd16834d"
+    (path "/fabbdae9-6a23-4e5a-893f-65c7010c9eb5/b1183543-3f60-49a5-acfa-37a9fabbb5e5"
       (reference "U1") (unit 1) (value "TL074") (footprint "Package_SO:SOIC-14_3.9x8.7mm_P1.27mm")
     )
@@
       (reference "U1") (unit 2) (value "TL074") (footprint "Package_SO:SOIC-14_3.9x8.7mm_P1.27mm")
     )
+    (path "/1c9013f3-dc47-4074-b623-b743c64985e1/e0a84abb-9577-4377-ad97-14afdd16834d"
+      (reference "U1") (unit 3) (value "TL074") (footprint "Package_SO:SOIC-14_3.9x8.7mm_P1.27mm")
+    )
     (path "/350871e3-5ee1-4577-9ae3-8c84468cb1f5"
-      (reference "U1") (unit 3) (value "TL074") (footprint "Package_SO:SOIC-14_3.9x8.7mm_P1.27mm")
-    )
-    (path "/fabbdae9-6a23-4e5a-893f-65c7010c9eb5/b1183543-3f60-49a5-acfa-37a9fabbb5e5"
       (reference "U1") (unit 4) (value "TL074") (footprint "Package_SO:SOIC-14_3.9x8.7mm_P1.27mm")
     )
@@
       (reference "U1") (unit 5) (value "TL074") (footprint "Package_SO:SOIC-14_3.9x8.7mm_P1.27mm")
     )
+    (path "/1c9013f3-dc47-4074-b623-b743c64985e1/00760eaf-801f-43a3-a2c1-e13ee21a87cc"
+      (reference "U2") (unit 1) (value "TL074") (footprint "Package_SO:SOIC-14_3.9x8.7mm_P1.27mm")
+    )
     (path "/1c9013f3-dc47-4074-b623-b743c64985e1/d1982675-d26f-453f-b6e7-1b38ce346730"
-      (reference "U2") (unit 1) (value "TL074") (footprint "Package_SO:SOIC-14_3.9x8.7mm_P1.27mm")
-    )
-    (path "/1c9013f3-dc47-4074-b623-b743c64985e1/00760eaf-801f-43a3-a2c1-e13ee21a87cc"
       (reference "U2") (unit 2) (value "TL074") (footprint "Package_SO:SOIC-14_3.9x8.7mm_P1.27mm")
     )
+    (path "/1c9013f3-dc47-4074-b623-b743c64985e1/ef0194b7-acc5-4bdd-b867-7a20113ce3be"
+      (reference "U2") (unit 3) (value "TL074") (footprint "Package_SO:SOIC-14_3.9x8.7mm_P1.27mm")
+    )
     (path "/1c9013f3-dc47-4074-b623-b743c64985e1/9e25b776-d83d-4899-9cdc-1ad2a02d8e60"
-      (reference "U2") (unit 3) (value "TL074") (footprint "Package_SO:SOIC-14_3.9x8.7mm_P1.27mm")
-    )
-    (path "/1c9013f3-dc47-4074-b623-b743c64985e1/ef0194b7-acc5-4bdd-b867-7a20113ce3be"
       (reference "U2") (unit 4) (value "TL074") (footprint "Package_SO:SOIC-14_3.9x8.7mm_P1.27mm")
     )

Commit message: Mouser parts ordered
Parts:
- C1: Mouser (none) -> 598-107SML016M
- U1: Mouser (none) -> 595-TL074IDR
Changed lines of the file:
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@@
+      (effects (font (size 1.27 1.27)) hide)
+    )
+    (property "Mouser" "595-TL074IDR" (id 4) (at 119.38 175.26 0)
       (effects (font (size 1.27 1.27)) hide)
     )
@@
       (effects (font (size 1.27 1.27)) hide)
     )
+    (property "Mouser" "598-107SML016M" (id 5) (at 71.12 177.8 0)
+      (effects (font (size 1.27 1.27)) hide)
+    )

Commit message: rev2 wip start
Parts:
- added Q?: MMBT3904, Package_TO_SOT_SMD:SOT-23, symbol Transistor_BJT:MMBT3904
- added R? (x2): 10k, symbol Device:R
- added R?: 1M, symbol Device:R
- added SW?: SW_SPST, symbol Switch:SW_SPST
Connections:
- net +9V: now also R?.1, R?.1
- net GND: now also Q?.2 (E), SW?.1 (A)
- net MomSw1: now also Q?.3 (C), R?.2
- new net: Q?.1 (B), R?.2, R?.2
- new net: R?.1, SW?.2 (B)
Other:
- note added: "Alt Mom switch"
- note added: "For rev.2: R24 & R25 = 10k Phase Sw (Sw1): invert pins"
Changed lines of the file:
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@@
   (junction (at 35.56 175.26) (diameter 0) (color 0 0 0 0)
   )
+  (junction (at 190.5 127) (diameter 0) (color 0 0 0 0)
+  )
   (junction (at 127 175.26) (diameter 0) (color 0 0 0 0)
   )
   (junction (at 71.12 166.37) (diameter 0) (color 0 0 0 0)
   )
+  (junction (at 190.5 138.43) (diameter 0) (color 0 0 0 0)
+  )
   (junction (at 143.51 175.26) (diameter 0) (color 0 0 0 0)
   )
+  (junction (at 182.88 144.78) (diameter 0) (color 0 0 0 0)
+  )
   (junction (at 46.99 166.37) (diameter 0) (color 0 0 0 0)
   )
@@
     (stroke (width 0) (type default) (color 0 0 0 0))
   )
+  (wire (pts (xy 182.88 134.62) (xy 182.88 144.78))
+    (stroke (width 0) (type default) (color 0 0 0 0))
+  )
   (wire (pts (xy 52.07 116.84) (xy 54.61 116.84))
     (stroke (width 0) (type default) (color 0 0 0 0))
@@
     (stroke (width 0) (type default) (color 0 0 0 0))
   )
+  (wire (pts (xy 190.5 138.43) (xy 203.2 138.43))
+    (stroke (width 0) (type default) (color 0 0 0 0))
+  )
+  (wire (pts (xy 167.64 144.78) (xy 171.45 144.78))
+    (stroke (width 0) (type default) (color 0 0 0 0))
+  )
   (wire (pts (xy 46.99 166.37) (xy 54.61 166.37))
     (stroke (width 0) (type default) (color 0 0 0 0))
@@
     (stroke (width 0) (type default) (color 0 0 0 0))
   )
+  (wire (pts (xy 179.07 144.78) (xy 182.88 144.78))
+    (stroke (width 0) (type default) (color 0 0 0 0))
+  )
   (wire (pts (xy 35.56 173.99) (xy 35.56 175.26))
     (stroke (width 0) (type default) (color 0 0 0 0))
   )
+  (wire (pts (xy 190.5 149.86) (xy 190.5 152.4))
+    (stroke (width 0) (type default) (color 0 0 0 0))
+  )
   (wire (pts (xy 114.3 73.025) (xy 117.475 73.025))
     (stroke (width 0) (type default) (color 0 0 0 0))
@@
     (stroke (width 0) (type default) (color 0 0 0 0))
   )
+  (wire (pts (xy 190.5 134.62) (xy 190.5 138.43))
+    (stroke (width 0) (type default) (color 0 0 0 0))
+  )
   (wire (pts (xy 68.58 166.37) (xy 71.12 166.37))
     (stroke (width 0) (type default) (color 0 0 0 0))
@@
     (stroke (width 0) (type default) (color 0 0 0 0))
   )
+  (wire (pts (xy 190.5 124.46) (xy 190.5 127))
+    (stroke (width 0) (type default) (color 0 0 0 0))
+  )
   (wire (pts (xy 127 175.26) (xy 129.54 175.26))
     (stroke (width 0) (type default) (color 0 0 0 0))
@@
     (stroke (width 0) (type default) (color 0 0 0 0))
   )
+  (wire (pts (xy 182.88 127) (xy 190.5 127))
+    (stroke (width 0) (type default) (color 0 0 0 0))
+  )
   (wire (pts (xy 52.07 114.3) (xy 54.61 114.3))
     (stroke (width 0) (type default) (color 0 0 0 0))
@@
     (stroke (width 0) (type default) (color 0 0 0 0))
   )
+  (wire (pts (xy 190.5 138.43) (xy 190.5 139.7))
+    (stroke (width 0) (type default) (color 0 0 0 0))
+  )
   (wire (pts (xy 204.47 55.88) (xy 212.09 55.88))
     (stroke (width 0) (type default) (color 0 0 0 0))
@@
     (stroke (width 0) (type default) (color 0 0 0 0))
   )
+  (wire (pts (xy 152.4 144.78) (xy 157.48 144.78))
+    (stroke (width 0) (type default) (color 0 0 0 0))
+  )
   (wire (pts (xy 143.51 175.26) (xy 143.51 177.8))
     (stroke (width 0) (type default) (color 0 0 0 0))
@@
     (stroke (width 0) (type default) (color 0 0 0 0))
   )
+  (text "For rev.2:\nR24 & R25 = 10k\nPhase Sw (Sw1): invert pins"
+    (at 176.53 89.535 0)
+    (effects (font (size 1.27 1.27) italic) (justify left bottom))
+  )
+  (text "Alt Mom switch" (at 176.53 104.775 0)
+    (effects (font (size 1.27 1.27)) (justify left bottom))
+  )
   (label "GND" (at 35.56 186.69 270)
     (effects (font (size 1.27 1.27)) (justify right bottom))
@@
     (effects (font (size 1.27 1.27)) (justify right bottom))
   )
+  (label "GND" (at 190.5 152.4 270)
+    (effects (font (size 1.27 1.27)) (justify right bottom))
+  )
   (label "+4V5" (at 59.69 47.625 90)
     (effects (font (size 1.27 1.27)) (justify left bottom))
@@
     (effects (font (size 1.27 1.27)) (justify right bottom))
   )
+  (label "+9V" (at 190.5 124.46 90)
+    (effects (font (size 1.27 1.27)) (justify left bottom))
+  )
   (label "+4V5" (at 166.37 175.26 0)
     (effects (font (size 1.27 1.27)) (justify left bottom))
@@
     (effects (font (size 1.27 1.27)) (justify left bottom))
   )
+  (label "GND" (at 152.4 144.78 270)
+    (effects (font (size 1.27 1.27)) (justify right bottom))
+  )
   (label "GND" (at 143.51 189.23 270)
     (effects (font (size 1.27 1.27)) (justify right bottom))
@@
   )
   (label "LatchSw2" (at 117.475 73.025 0)
+    (effects (font (size 1.27 1.27)) (justify left bottom))
+  )
+  (label "MomSw1" (at 203.2 138.43 0)
     (effects (font (size 1.27 1.27)) (justify left bottom))
   )
@@
     )
     (pin "1")
+  )
+  (symbol (lib_id "Device:R") (at 190.5 130.81 0) (unit 1)
+    (in_bom yes) (on_board yes) (fields_autoplaced)
+    (property "Reference" "R?" (id 0) (at 193.04 129.5399 0)
+      (effects (font (size 1.27 1.27)) (justify left))
+    )
+    (property "Value" "10k" (id 1) (at 193.04 132.0799 0)
+      (effects (font (size 1.27 1.27)) (justify left))
+    )
+    (property "Footprint" "" (id 2) (at 188.722 130.81 90)
+      (effects (font (size 1.27 1.27)) hide)
+    )
+    (property "Datasheet" "~" (id 3) (at 190.5 130.81 0)
+      (effects (font (size 1.27 1.27)) hide)
+    )
+    (pin "1")
+    (pin "2")
   )
   (symbol (lib_id "Diode:1N4148") (at 41.91 175.26 180) (unit 1)
@@
     (pin "1")
   )
+  (symbol (lib_id "Transistor_BJT:MMBT3904") (at 187.96 144.78 0) (unit 1)
+    (in_bom yes) (on_board yes) (fields_autoplaced)
+    (property "Reference" "Q?" (id 0) (at 193.04 143.5099 0)
+      (effects (font (size 1.27 1.27)) (justify left))
+    )
+    (property "Value" "MMBT3904" (id 1) (at 193.04 146.0499 0)
+      (effects (font (size 1.27 1.27)) (justify left))
+    )
+    (property "Footprint" "Package_TO_SOT_SMD:SOT-23" (id 2) (at 193.04 146.685 0)
+      (effects (font (size 1.27 1.27) italic) (justify left) hide)
+    )
+    (property "Datasheet" "https://www.onsemi.com/pub/Collateral/2N3903-D.PDF" (id 3) (at 187.96 144.78 0)
+      (effects (font (size 1.27 1.27)) (justify left) hide)
+    )
+    (pin "1")
+    (pin "2")
+    (pin "3")
+  )
   (symbol (lib_id "Connector:Conn_01x02_Male") (at 101.6 114.3 0) (mirror y) (unit 1)
     (in_bom yes) (on_board yes) (fields_autoplaced)
@@
     )
     (property "Datasheet" "~" (id 3) (at 101.6 114.3 0)
+      (effects (font (size 1.27 1.27)) hide)
+    )
+    (pin "1")
+    (pin "2")
+  )
+  (symbol (lib_id "Switch:SW_SPST") (at 162.56 144.78 0) (unit 1)
+    (in_bom yes) (on_board yes) (fields_autoplaced)
+    (property "Reference" "SW?" (id 0) (at 162.56 138.43 0))
+    (property "Value" "SW_SPST" (id 1) (at 162.56 140.97 0))
+    (property "Footprint" "" (id 2) (at 162.56 144.78 0)
+      (effects (font (size 1.27 1.27)) hide)
+    )
+    (property "Datasheet" "~" (id 3) (at 162.56 144.78 0)
       (effects (font (size 1.27 1.27)) hide)
     )
@@
     )
     (property "Mouser" "710-865080440002" (id 6) (at 101.6 181.61 0)
+      (effects (font (size 1.27 1.27)) hide)
+    )
+    (pin "1")
+    (pin "2")
+  )
+  (symbol (lib_id "Device:R") (at 182.88 130.81 0) (unit 1)
+    (in_bom yes) (on_board yes) (fields_autoplaced)
+    (property "Reference" "R?" (id 0) (at 185.42 129.5399 0)
+      (effects (font (size 1.27 1.27)) (justify left))
+    )
+    (property "Value" "1M" (id 1) (at 185.42 132.0799 0)
+      (effects (font (size 1.27 1.27)) (justify left))
+    )
+    (property "Footprint" "" (id 2) (at 181.102 130.81 90)
+      (effects (font (size 1.27 1.27)) hide)
+    )
+    (property "Datasheet" "~" (id 3) (at 182.88 130.81 0)
       (effects (font (size 1.27 1.27)) hide)
     )
@@
     (pin "2")
   )
+  (symbol (lib_id "Device:R") (at 175.26 144.78 90) (unit 1)
+    (in_bom yes) (on_board yes) (fields_autoplaced)
+    (property "Reference" "R?" (id 0) (at 175.26 138.43 90))
+    (property "Value" "10k" (id 1) (at 175.26 140.97 90))
+    (property "Footprint" "" (id 2) (at 175.26 146.558 90)
+      (effects (font (size 1.27 1.27)) hide)
+    )
+    (property "Datasheet" "~" (id 3) (at 175.26 144.78 0)
+      (effects (font (size 1.27 1.27)) hide)
+    )
+    (pin "1")
+    (pin "2")
+  )
   (symbol (lib_id "Device:C") (at 154.94 181.61 180) (unit 1)
     (in_bom yes) (on_board yes) (fields_autoplaced)
@@
       (reference "Q4") (unit 1) (value "MMBT3904") (footprint "Package_TO_SOT_SMD:SOT-23")
     )
+    (path "/5408cb3a-e1a6-4dbe-9c88-56bc00addc2f"
+      (reference "Q?") (unit 1) (value "MMBT3904") (footprint "Package_TO_SOT_SMD:SOT-23")
+    )
     (path "/9eb9cc92-310b-4809-b5ba-53b51310f663"
       (reference "R1") (unit 1) (value "1M") (footprint "Resistor_SMD:R_0603_1608Metric_Pad0.98x0.95mm_HandSolder")
@@
       (reference "R39") (unit 1) (value "100k") (footprint "Resistor_SMD:R_0603_1608Metric_Pad0.98x0.95mm_HandSolder")
     )
+    (path "/14523acd-5dd4-4b86-8145-1c3d1c811a92"
+      (reference "R?") (unit 1) (value "10k") (footprint "")
+    )
+    (path "/8182bc7e-3dd8-4e3a-94ab-980a36146f0e"
+      (reference "R?") (unit 1) (value "1M") (footprint "")
+    )
+    (path "/d2fbc276-164c-42d6-9dae-a33dcd454874"
+      (reference "R?") (unit 1) (value "10k") (footprint "")
+    )
     (path "/1c9013f3-dc47-4074-b623-b743c64985e1/800e6ec3-9175-4513-9bb2-e8f7f441d8b6"
       (reference "RV1") (unit 1) (value "A10k") (footprint "Pots:V3_TRIM_R0904NB10KL-Keepout")
@@
       (reference "SW2") (unit 1) (value "SW_SPDT") (footprint "MBP switches:SPDT.LUGS.PM")
     )
+    (path "/58c01ec3-66e2-4ebe-9fac-a820b3caa5f3"
+      (reference "SW?") (unit 1) (value "SW_SPST") (footprint "")
+    )
     (path "/fabbdae9-6a23-4e5a-893f-65c7010c9eb5/b1183543-3f60-49a5-acfa-37a9fabbb5e5"

Commit message: Wip rev2
Parts:
- removed Q?: MMBT3904, Package_TO_SOT_SMD:SOT-23, symbol Transistor_BJT:MMBT3904
- removed R? (x2): 10k, symbol Device:R
- removed R?: 1M, symbol Device:R
- removed SW?: SW_SPST, symbol Switch:SW_SPST
- added R31: 10k, Resistor_SMD:R_0603_1608Metric_Pad0.98x0.95mm_HandSolder, symbol Device:R
Connections:
- net +9V: now also R31.2; no longer J2.2 (Pin_2)
- new net: J2.2 (Pin_2), R31.1
Other:
- note added: "For rev.2: v R24 & R25 = 10k v Phase Sw (Sw1): invert pins"
- note removed: "Alt Mom switch"
- note removed: "For rev.2: R24 & R25 = 10k Phase Sw (Sw1): invert pins"
