File: feedback-main-board/feedback-main-board.kicad_sch (KiCad schematic)
At the start: 15 parts, among them J1 908140508, J2 FLIP, J3 RPT, Q1 MMFTP3401, U1 OPA1679

Commit message: Main rev4 ordered
Parts:
- added R42: 10, Resistor_SMD:R_0603_1608Metric_Pad0.98x0.95mm_HandSolder, symbol Device:R
- C1: LCSC DNP -> C2836437
- C2, C3: value 10u -> 22u; LCSC DNP -> C23289; Mouser 710-865080440002 -> (none)
- R4: value 10 -> 0; LCSC C22859 -> C21189
Connections:
- net at R4.1, U1.13 (-): now also R42.2; no longer U1.14
- new net: R42.1, U1.14
Other:
- note removed: "For rev.2: v R24 & R25 = 10k v Phase Sw (Sw1): invert pins"
- moved on the sheet: C3, C4, R4, U1D
