File: feedback-main-board/feedback-main-board.kicad_sch (KiCad schematic)
At the start: 15 parts, among them J1 908140508, J2 FLIP, J3 RPT, Q1 MMFTP3401, U1 TL074

Commit message: rev4
Parts:
- added R42: 10, Resistor_SMD:R_0603_1608Metric_Pad0.98x0.95mm_HandSolder, symbol Device:R
- C1: LCSC C4747963 -> C2836437
- C2, C3: value 10u -> 22u; LCSC C294524 -> C23289; Mouser 710-865080440002 -> (none)
- C4: LCSC (none) -> C14663; Mouser (none) -> 581-06035C105MAT2A
- D1: LCSC (none) -> C6423741
- J1, J2, J3: LCSC (none) -> DNP
- Q1: LCSC (none) -> C596234
- R1: LCSC (none) -> C22935
- R2, R3: value 10K -> 10k; LCSC (none) -> C25804
- R31: LCSC (none) -> C25804
- R4: value 10 -> 0; LCSC (none) -> C21189
- U1: value TL074 -> OPA1679; LCSC (none) -> C2878631; Mouser 595-TL074IDR -> (none)
Connections:
- net at R4.1, U1.13 (-): now also R42.2; no longer U1.14
- new net: R42.1, U1.14
Other:
- note removed: "For rev.2: v R24 & R25 = 10k v Phase Sw (Sw1): invert pins"
- moved on the sheet: C3, C4, R4, U1D
