File: feedback-main-board/feedback-main-board.kicad_sch (KiCad schematic)
At the start: 16 parts, among them J1 908140508, J2 FLIP, J3 RPT, Q1 MMFTP3401, U1 OPA1679

Commit message: wip
Parts:
- removed J1: 908140508, molex-picoflex8:CONN_SDA-90814_08_MOL, symbol molex-picoflex8:908140508
- added J1: FPC_Connector, Connector_FFC-FPC:JUSHUO_AFA07-S08FCA-00_1x8-1MP_P1.0mm_Horizontal, symbol Connector_Generic_MountingPin:Conn_01x08_MountingPin
- added JP? (x2): Jumper_2_Bridged, symbol Jumper:Jumper_2_Bridged
- C2, C3: value 22u -> 47u; LCSC C23289 -> C4747958
- J2, J3: now not fitted
Connections:
- net GND: now also J1.2 (Pin_2), J1.5 (Pin_5), J1.8 (Pin_8), JP?.1 (A), JP?.1 (A); no longer C1.2, C2.2, C3.2, C4.1, R1.1, R3.2
- net In: now also J1.3 (Pin_3)
- net Jack9V: now also J1.1 (Pin_1)
- net Out: now also J1.7 (Pin_7)
- net Ret: now also J1.6 (Pin_6)
- net Snd: now also J1.4 (Pin_4)
- new net PWR_GND: JP?.2 (B), R1.1
- new net SIG_GND: C1.2, C2.2, C3.2, C4.1, J1.MP (MountPin), JP?.2 (B), R3.2
Other:
- sheet Core ports: added PWR_GND, SIG_GND; removed GND

Commit message: wip
Parts:
- removed JP? (x2): Jumper_2_Bridged, symbol Jumper:Jumper_2_Bridged
Connections:
- net PWR_GND is gone; now on net GND: R1.1
- net SIG_GND is gone; now on net GND: C1.2, C2.2, C3.2, C4.1, J1.MP (MountPin), R3.2
Other:
- sheet Core ports: added GND; removed PWR_GND, SIG_GND

Commit message: wip pre grouping jfets
Parts:
- D1: LCSC C6423741 -> C2128
Changed lines of the file:
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@@
 			)
 		)
-		(property "LCSC" "C6423741"
+		(property "LCSC" "C2128"
 			(at 41.91 175.26 0)
 			(hide yes)

Commit message: wip jacks board
Other:
- company: Pedal Markt / Andrei Salomatin -> Andrei Salomatin / akkusativ
- title: Read/Repeat -> RDRPT
- moved on the sheet: J2, R4, R42, U1D
