File: feedback-main-board/feedback-main-board.kicad_pcb (KiCad board)
At the start: 4 copper layers, 80 x 64 mm, 101 parts, among them J1 908140508, J2 FLIP, J3 RPT, Q1 MMFTP3401, Q2 MMBT3904, Q3 MMBT3904, Q4 MMBT3904, SW1 SW_SPDT, SW2 SW_SPDT, U1 TL074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

Commit message: rev2 main board layout getting close
Parts:
- removed C22: 100n, Capacitor_SMD:C_0603_1608Metric_Pad1.08x0.95mm_HandSolder
- removed U5: 4070, Package_SO:SOIC-14_3.9x8.7mm_P1.27mm
- removed kibuzzard-67A4ED41: G***, kibuzzard-67A4ED41
- added Q5: MMBT3904, Package_TO_SOT_SMD:SOT-23, B.Cu at (110.1, 106.9)
- added R42: 100k, Resistor_SMD:R_0603_1608Metric_Pad0.98x0.95mm_HandSolder, B.Cu at (98.3, 116.1)
- added kibuzzard-67BCC318: G***, kibuzzard-67BCC318, B.Cu at (100.0, 133.5)
- C12, C13, C7, C8, C9: value 2u2 -> 1u; footprint Capacitor_THT:C_Rect_L7.2mm_W7.2mm_P5.00mm_FKS2_FKP2_MKS2_MKP2 -> Capacitor_THT:C_Rect_L7.0mm_W4.5mm_P5.00mm
- C23, C24: value 100n -> 1u; footprint Capacitor_THT:C_Rect_L7.0mm_W2.5mm_P5.00mm -> Capacitor_THT:C_Rect_L7.0mm_W4.5mm_P5.00mm
- R12, R20, R22, R23: value 10k -> 100k
- RV1, RV2, RV3: value A10k -> A100k
- U3: value DG403 -> TMUX4053; footprint Package_SO:SOIC-16_3.9x9.9mm_P1.27mm -> Package_SO:TSSOP-16_4.4x5mm_P0.65mm
- U4: value NE555P -> NE555
- moved R30 38.7 mm to (110.1, 111.8)
- moved R23 13.1 mm to (101.1, 106.9), turned to -90 degrees
- moved U4 8.64 mm to (67.9, 120.7)
- moved R22 8.46 mm to (103.9, 106.9), turned to -90 degrees
- moved R32 4.04 mm to (106.4, 106.9), turned to -90 degrees
- moved C17 3.90 mm to (65.5, 115.8), turned to 90 degrees
- moved R31 3.02 mm to (77.0, 128.4), turned to -90 degrees
- moved C21 2.95 mm to (98.4, 111.8)
- moved R20 2.79 mm to (98.3, 106.9)
- moved C6 1.40 mm to (94.4, 110.1)
- moved R1 1.20 mm to (73.4, 123.7)
- moved D1 1.17 mm to (77.0, 119.5)
- moved Q1 1.02 mm to (77.0, 124.0)
- moved R33 1.02 mm to (136.9, 132.8)
- moved C12 0.51 mm to (89.4, 116.2)
Connections:
- C13 pad 2: Net-(C13-Pad2) -> /Core/FeedbackClip
- C20 pad 1: /MomSw1 -> /MomSw2
- C23 pad 1: Net-(R22-Pad2) -> Net-(C23-Pad1)
- C24 pad 1: Net-(R23-Pad2) -> Net-(C24-Pad1)
- J2 pad 2: Net-(R31-Pad1) -> /MomSw2
- R22 pad 2: Net-(R22-Pad2) -> Net-(C23-Pad1)
- R23 pad 2: Net-(R23-Pad2) -> Net-(C24-Pad1)
- R30 pad 1: Net-(R30-Pad1) -> /Switching/LatchState
- R30 pad 2: /Switching/LatchState -> Net-(Q5-Pad1)
- R31 pad 1: Net-(R31-Pad1) -> /+9V
- R31 pad 2: /+9V -> /MomSw1
- R32 pad 1: /Switching/BypassState -> /Switching/~{LatchState}
- R32 pad 2: Net-(R32-Pad2) -> /+9V
- R35 pad 1: /MomSw1 -> /MomSw2
- R39 pad 1: /MomSw1 -> /MomSw2
- RV3 pad 3: Net-(C13-Pad2) -> /Core/FeedbackClip
- SW2 pad 3: /Core/Feedback -> /Core/FeedbackClip
- U3 pad 1: Net-(R22-Pad2) -> /Core/FxOut
- U3 pad 11: /+9V -> /Switching/BypassState
- U3 pad 12: /+9V -> /Core/InBuf
- U3 pad 13: /+4V5 -> /Core/Sum
- U3 pad 14: /GND -> Net-(C23-Pad1)
- U3 pad 15: /Switching/BypassState -> Net-(C24-Pad1)
- U3 pad 16: /Core/Sum -> /+9V
- U3 pad 2: (no net) -> /Core/RetBuf
- U3 pad 3: Net-(R22-Pad2) -> /Switching/~{LatchState}
- U3 pad 4: /Core/InBuf -> /Switching/BypassState
- U3 pad 5: /Core/RetBuf -> /Switching/LatchState
- U3 pad 6: Net-(R23-Pad2) -> /GND
- U3 pad 7: (no net) -> /GND
- U3 pad 8: Net-(R23-Pad2) -> /GND
- U3 pad 9: /Core/FxOut -> /MomSw2
Routing:
- net /MomSw2: track 0.00 -> 62.6 mm, vias 0 -> 4
- net Net-(R32-Pad2): track 59.5 -> 0.00 mm, vias 2 -> 0
- net Net-(C23-Pad1): track 0.00 -> 54.7 mm
- net /Switching/LatchState: track 94.3 -> 141.7 mm, vias 2 -> 3
- net /Core/FeedbackClip: track 0.00 -> 46.7 mm, vias 0 -> 1
- net Net-(C24-Pad1): track 0.00 -> 40.9 mm
- net Net-(R22-Pad2): track 34.4 -> 0.00 mm
- net /MomSw1: track 35.9 -> 4.14 mm
- net /Core/Feedback: track 50.3 -> 20.7 mm
- net /+9V: track 244.8 -> 268.9 mm, vias 14 -> 13
- net Net-(R23-Pad2): track 22.9 -> 0.00 mm
- net /GND: track 109.5 -> 93.8 mm, vias 84 -> 88
- net Net-(C13-Pad2): track 15.0 -> 0.00 mm
- net /Switching/BypassState: track 62.8 -> 77.0 mm
- net /Switching/~{LatchState}: track 0.00 -> 11.6 mm
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
Commit message: Jack board updates
Routing:
- net /GND: track 93.8 -> 109.7 mm, vias 88 -> 85
- net /+4V5: vias 32 -> 34
