File: feedback-main-board/feedback-main-board.kicad_pcb (KiCad board)
At the start: 4 copper layers, 80 x 64 mm, 101 parts, among them J1 908140508, J2 FLIP, J3 RPT, Q1 MMFTP3401, Q2 MMBT3904, Q3 MMBT3904, Q4 MMBT3904, SW1 SW_SPDT, SW2 SW_SPDT, U1 TL074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

Commit message: Changes pre-rev3
Parts:
- removed kibuzzard-67A4ED41: G***, kibuzzard-67A4ED41
- added kibuzzard-67D43B6A: G***, kibuzzard-67D43B6A, B.Cu at (100.0, 133.5)
- C20: value 1u -> 100n
- R2, R3: value 10K -> 10k
- U4: value NE555P -> NE555
- U5: value 4070 -> CD4070
- moved R32 12.0 mm to (98.3, 105.8), turned to -90 degrees
- turned R27 to 90 degrees
Connections:
- C13 pad 2: Net-(C13-Pad2) -> /Core/PreFeedback
- RV3 pad 3: Net-(C13-Pad2) -> /Core/PreFeedback
- SW2 pad 3: /Core/Feedback -> /Core/PreFeedback
- U3 pad 13: /+4V5 -> /GND
Routing:
- net /Core/PreFeedback: track 0.00 -> 42.6 mm
- net Net-(R32-Pad2): track 59.5 -> 39.4 mm
- net /Core/Feedback: track 50.3 -> 33.5 mm
- net Net-(C13-Pad2): track 15.0 -> 0.00 mm
- net /LatchSw1: track 61.7 -> 75.5 mm, vias 5 -> 2
- net /Switching/BypassState: track 62.8 -> 51.0 mm, vias 4 -> 2
- net Net-(C19-Pad1): track 44.8 -> 38.4 mm
- net Net-(C24-Pad2): track 52.9 -> 47.1 mm, vias 4 -> 2
- net Net-(C18-Pad1): track 28.0 -> 24.9 mm
- net /+4V5: track 14.6 -> 17.7 mm, vias 31 -> 32
- net /GND: track 109.5 -> 111.6 mm, vias 84 -> 77
- net /Core/RetBuf: track 80.5 -> 78.6 mm
- net Net-(R27-Pad1): track 5.26 -> 4.52 mm
- net /Snd: track 39.9 -> 40.5 mm
- net /Core/FxOut: track 113.9 -> 113.3 mm, vias 4 -> 2
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
Commit message: JLCPCB rev3 ordered
Parts:
- C23, C24: value 100n -> 1u
- U1, U2: value TL074 -> OPA1679
Other:
- board text added: "JLCJLCJLCJLC"
Changed lines of the file:
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@@
     (fp_line (start 4.95 2.35) (end -2.45 2.35) (layer "B.Fab") (width 0.1))
     (fp_line (start 4.95 -3.4) (end 4.95 2.35) (layer "B.Fab") (width 0.1))
-    (pad "1" thru_hole roundrect locked (at 0 0) (size 1.7 2) (drill 1) (layers *.Cu *.Mask) (roundrect_rratio 0.147059)
+    (pad "1" thru_hole roundrect locked (at 0 0) (size 1.7 2) (drill 1) (layers *.Cu *.Mask) (roundrect_rratio 0.1470588235)
       (net 39 "/MomSw1") (pinfunction "Pin_1") (pintype "passive"))
     (pad "2" thru_hole oval locked (at 2.5 0) (size 1.7 2) (drill 1) (layers *.Cu *.Mask)
@@
     (fp_line (start 4.95 -3.4) (end 4.95 2.35) (layer "B.Fab") (width 0.1))
     (fp_line (start 4.95 2.35) (end -2.45 2.35) (layer "B.Fab") (width 0.1))
-    (pad "1" thru_hole roundrect locked (at 0 0) (size 1.7 2) (drill 1) (layers *.Cu *.Mask) (roundrect_rratio 0.147059)
+    (pad "1" thru_hole roundrect locked (at 0 0) (size 1.7 2) (drill 1) (layers *.Cu *.Mask) (roundrect_rratio 0.1470588235)
       (net 50 "/LatchSw1") (pinfunction "Pin_1") (pintype "passive"))
     (pad "2" thru_hole oval locked (at 2.5 0) (size 1.7 2) (drill 1) (layers *.Cu *.Mask)
@@
     (descr "SOIC, 14 Pin (JEDEC MS-012AB, https://www.analog.com/media/en/package-pcb-resources/package/pkg_pdf/soic_narrow-r/r_14.pdf), generated with kicad-footprint-generator ipc_gullwing_generator.py")
     (tags "SOIC SO")
-    (property "LCSC" "C6964")
-    (property "Mouser" "595-TL074IDR")
+    (property "LCSC" "C2878631")
+    (property "Mouser" "")
     (property "Sheetfile" "core.kicad_sch")
     (property "Sheetname" "Core")
@@
       (effects (font (size 1 1) (thickness 0.15)) (justify mirror))
     )
-    (fp_text value "TL074" (at 0 -5.28) (layer "B.Fab")
+    (fp_text value "OPA1679" (at 0 -5.28) (layer "B.Fab")
       (effects (font (size 1 1) (thickness 0.15)) (justify mirror))
     )
@@
       (effects (font (size 1 1) (thickness 0.15)) (justify mirror))
     )
-    (fp_text value "100n" (at 2.5 -2.5) (layer "B.Fab")
+    (fp_text value "1u" (at 2.5 -2.5) (layer "B.Fab")
       (effects (font (size 1 1) (thickness 0.15)) (justify mirror))
     )
@@
       (effects (font (size 1 1) (thickness 0.15)) (justify mirror))
     )
-    (fp_text value "100n" (at 2.5 -2.5) (layer "B.Fab")
+    (fp_text value "1u" (at 2.5 -2.5) (layer "B.Fab")
       (effects (font (size 1 1) (thickness 0.15)) (justify mirror))
     )
@@
     (attr board_only exclude_from_pos_files exclude_from_bom)
     (fp_text reference "kibuzzard-67D43B6A" (at 0 3.572669) (layer "B.SilkS") hide
-      (effects (font (size 0 0)) (justify mirror))
+      (effects (font (size 0 0) (thickness 0.15)) (justify mirror))
     )
     (fp_text value "G***" (at 0 -3.572669) (layer "B.SilkS") hide
-      (effects (font (size 0 0)) (justify mirror))
+      (effects (font (size 0 0) (thickness 0.15)) (justify mirror))
     )
     (fp_poly (pts
@@
     (descr "SOIC, 14 Pin (JEDEC MS-012AB, https://www.analog.com/media/en/package-pcb-resources/package/pkg_pdf/soic_narrow-r/r_14.pdf), generated with kicad-footprint-generator ipc_gullwing_generator.py")
     (tags "SOIC SO")
-    (property "LCSC" "C6964")
-    (property "Mouser" "595-TL074IDR")
+    (property "LCSC" "C2878631")
+    (property "Mouser" "")
     (property "Sheetfile" "feedback-main-board.kicad_sch")
     (property "Sheetname" "")
@@
       (effects (font (size 1 1) (thickness 0.15)) (justify mirror))
     )
-    (fp_text value "TL074" (at 0 -5.28) (layer "B.Fab")
+    (fp_text value "OPA1679" (at 0 -5.28) (layer "B.Fab")
       (effects (font (size 1 1) (thickness 0.15)) (justify mirror))
     )
@@
   (gr_rect locked (start 56.5 44) (end 143.5 156) (layer "User.8") (width 0.15) (fill none))
   (gr_rect locked (start 54.5 42) (end 145.5 158) (layer "User.8") (width 0.15) (fill none))
+  (gr_text "JLCJLCJLCJLC" (at 99.949 91.821) (layer "F.SilkS")
+    (effects (font (size 0.8 0.8) (thickness 0.15)))
+  )
   (segment (start 131.457 97.651) (end 123.94 97.651) (width 0.5) (layer "F.Cu") (net 1))
   (segment (start 101.727 117.856) (end 105.156 117.856) (width 0.5) (layer "F.Cu") (net 1))

Commit message: Main rev4 ordered
Parts:
- removed kibuzzard-67D43B6A: G***, kibuzzard-67D43B6A
- added R42: 10, Resistor_SMD:R_0603_1608Metric_Pad0.98x0.95mm_HandSolder, B.Cu at (128.7, 90.4)
- added kibuzzard-682B2F26: G***, kibuzzard-682B2F26, B.Cu at (100.0, 133.5)
- C2, C3: value 10u -> 22u
- R4: value 10 -> 0
Connections:
- R4 pad 1: Net-(R4-Pad1) -> Net-(U1-Pad13)
- U1 pad 13: Net-(R4-Pad1) -> Net-(U1-Pad13)
- U1 pad 14: Net-(R4-Pad1) -> Net-(U1-Pad14)
Routing:
- net Net-(U1-Pad13): track 0.00 -> 21.9 mm
- net Net-(R4-Pad1): track 18.6 -> 0.00 mm
- net Net-(U1-Pad14): track 0.00 -> 1.78 mm
- net Net-(C19-Pad1): track 38.4 -> 37.7 mm
