File: feedback-main-board/feedback-main-board.kicad_pcb (KiCad board)
At the start: 4 copper layers, 80 x 64 mm, 101 parts, among them J1 908140508, J2 FLIP, J3 RPT, Q1 MMFTP3401, Q2 MMBT3904, Q3 MMBT3904, Q4 MMBT3904, SW1 SW_SPDT, SW2 SW_SPDT, U1 TL074, U2 TL074, U3 DG403, U4 NE555P, U5 4070

Commit message: rev4
Parts:
- removed kibuzzard-67A4ED41: G***, kibuzzard-67A4ED41
- added R42: 10, Resistor_SMD:R_0603_1608Metric_Pad0.98x0.95mm_HandSolder, B.Cu at (128.7, 90.4)
- added kibuzzard-682B2F26: G***, kibuzzard-682B2F26, B.Cu at (100.0, 133.5)
- C2, C3: value 10u -> 22u
- C20: value 1u -> 100n
- C23, C24: value 100n -> 1u
- R2, R3: value 10K -> 10k
- R4: value 10 -> 0
- U1, U2: value TL074 -> OPA1679
- U4: value NE555P -> NE555
- U5: value 4070 -> CD4070
- moved R32 12.0 mm to (98.3, 105.8), turned to -90 degrees
- turned R27 to 90 degrees
Connections:
- C13 pad 2: Net-(C13-Pad2) -> /Core/PreFeedback
- R4 pad 1: Net-(R4-Pad1) -> Net-(U1-Pad13)
- RV3 pad 3: Net-(C13-Pad2) -> /Core/PreFeedback
- SW2 pad 3: /Core/Feedback -> /Core/PreFeedback
- U1 pad 13: Net-(R4-Pad1) -> Net-(U1-Pad13)
- U1 pad 14: Net-(R4-Pad1) -> Net-(U1-Pad14)
- U3 pad 13: /+4V5 -> /GND
Routing:
- net /Core/PreFeedback: track 0.00 -> 42.6 mm
- net Net-(U1-Pad13): track 0.00 -> 21.9 mm
- net Net-(R32-Pad2): track 59.5 -> 39.4 mm
- net Net-(R4-Pad1): track 19.0 -> 0.00 mm
- net /Core/Feedback: track 50.3 -> 33.5 mm
- net Net-(C13-Pad2): track 15.0 -> 0.00 mm
- net /LatchSw1: track 61.7 -> 75.5 mm, vias 5 -> 2
- net /Switching/BypassState: track 62.8 -> 51.0 mm, vias 4 -> 2
- net Net-(C19-Pad1): track 44.8 -> 37.7 mm
- net Net-(C24-Pad2): track 52.9 -> 47.1 mm, vias 4 -> 2
- net Net-(C18-Pad1): track 28.0 -> 24.9 mm
- net /+4V5: track 14.6 -> 17.7 mm, vias 31 -> 32
- net /GND: track 109.5 -> 111.6 mm, vias 84 -> 77
- net /Core/RetBuf: track 80.5 -> 78.6 mm
- net Net-(U1-Pad14): track 0.00 -> 1.78 mm
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Other:
- board text added: "JLCJLCJLCJLC"

Commit message: wip pre grouping jfets
Parts:
- removed U3: DG403, Package_SO:SOIC-16_3.9x9.9mm_P1.27mm
- added C25: dnp, Capacitor_THT:C_Disc_D7.0mm_W2.5mm_P5.00mm, B.Cu at (109.1, 94.5)
- added C26: 47n, Capacitor_SMD:C_0603_1608Metric_Pad1.08x0.95mm_HandSolder, B.Cu at (119.4, 110.7)
- added C27: dnp, Capacitor_THT:C_Disc_D7.0mm_W2.5mm_P5.00mm, B.Cu at (122.2, 110.3)
- added C28: 47n, Capacitor_SMD:C_0603_1608Metric_Pad1.08x0.95mm_HandSolder, B.Cu at (75.4, 74.9)
- added C29: dnp, Capacitor_THT:C_Disc_D7.0mm_W2.5mm_P5.00mm, B.Cu at (71.3, 72.9)
- added C30: 47n, Capacitor_SMD:C_0603_1608Metric_Pad1.08x0.95mm_HandSolder, B.Cu at (92.7, 77.2)
- added C31: dnp, Capacitor_THT:C_Disc_D7.0mm_W2.5mm_P5.00mm, B.Cu at (88.8, 81.6)
- added C32: 47u, Capacitor_SMD:CP_Elec_5x5.4, B.Cu at (112.1, 82.3)
- added C33: 47u, Capacitor_SMD:CP_Elec_5x5.4, B.Cu at (82.8, 87.9)
- added C34: 47u, Capacitor_SMD:CP_Elec_5x5.4, B.Cu at (113.4, 104.8)
- added C35: 47u, Capacitor_SMD:CP_Elec_5x5.4, B.Cu at (120.5, 75.9)
- added C36: 47u, Capacitor_SMD:CP_Elec_5x5.4, B.Cu at (105.4, 120.7)
- added C37: 47u, Capacitor_SMD:CP_Elec_5x5.4, B.Cu at (92.5, 120.8)
- added D10: 1N4148, Diode_SMD:D_SOD-323_HandSoldering, B.Cu at (116.2, 110.9)
- added D11: 1N4148, Diode_SMD:D_SOD-323_HandSoldering, B.Cu at (80.8, 74.9)
- added D12: 1N4148, Diode_SMD:D_SOD-323_HandSoldering, B.Cu at (88.8, 85.9)
- added D9: 1N4148, Diode_SMD:D_SOD-323_HandSoldering, B.Cu at (111.8, 89.8)
- added Q5: MMBFJ201, Package_TO_SOT_SMD:SOT-23-3, B.Cu at (106.9, 85.7)
- added Q6: MMBFJ201, Package_TO_SOT_SMD:SOT-23-3, B.Cu at (125.1, 104.8)
- added Q7: MMBFJ201, Package_TO_SOT_SMD:SOT-23-3, B.Cu at (85.0, 74.9)
- added Q8: MMBFJ201, Package_TO_SOT_SMD:SOT-23-3, B.Cu at (92.7, 85.9)
- added R43: 1M, Resistor_SMD:R_0603_1608Metric_Pad0.98x0.95mm_HandSolder, B.Cu at (119.4, 114.8)
- added R44: 1M, Resistor_SMD:R_0603_1608Metric_Pad0.98x0.95mm_HandSolder, B.Cu at (96.5, 77.2)
- added R45: 1M, Resistor_SMD:R_0603_1608Metric_Pad0.98x0.95mm_HandSolder, B.Cu at (92.7, 81.2)
- added R46: 4.7k, Resistor_SMD:R_0603_1608Metric_Pad0.98x0.95mm_HandSolder, B.Cu at (119.4, 99.8)
- added R47: 4.7k, Resistor_SMD:R_0603_1608Metric_Pad0.98x0.95mm_HandSolder, B.Cu at (91.6, 104.0)
- added R48: 10k, Resistor_SMD:R_0603_1608Metric_Pad0.98x0.95mm_HandSolder, B.Cu at (119.4, 104.8)
- added R49: 10k, Resistor_SMD:R_0603_1608Metric_Pad0.98x0.95mm_HandSolder, B.Cu at (77.5, 89.4)
- added TP1: BypassOff, TestPoint:TestPoint_Pad_D1.5mm, B.Cu at (116.7, 115.7)
- added TP2: BypassOn, TestPoint:TestPoint_Pad_D1.5mm, B.Cu at (101.9, 92.5)
- added TP3: SigSwOut, TestPoint:TestPoint_Pad_D1.5mm, B.Cu at (106.0, 104.9)
- added TP4: SigSwOut, TestPoint:TestPoint_Pad_D1.5mm, B.Cu at (95.9, 88.1)
- C12, C13, C18, C19, C9: value 2u2 -> 47u; footprint Capacitor_THT:C_Rect_L7.2mm_W7.2mm_P5.00mm_FKS2_FKP2_MKS2_MKP2 -> Capacitor_SMD:CP_Elec_5x5.4
- C2, C3: value 22u -> 47u
- C21: value 100n -> 47n
- C23, C24: value 1u -> 47u; footprint Capacitor_THT:C_Rect_L7.0mm_W2.5mm_P5.00mm -> Capacitor_SMD:CP_Elec_5x5.4
- C5: footprint Capacitor_THT:C_Rect_L7.0mm_W2.5mm_P5.00mm -> Capacitor_SMD:C_1206_3216Metric_Pad1.33x1.80mm_HandSolder
- C6: value 1u -> 100n; footprint Capacitor_THT:C_Rect_L7.0mm_W4.5mm_P5.00mm -> Capacitor_SMD:C_1206_3216Metric_Pad1.33x1.80mm_HandSolder
- C7, C8: value 2u2 -> 220p; footprint Capacitor_THT:C_Rect_L7.2mm_W7.2mm_P5.00mm_FKS2_FKP2_MKS2_MKP2 -> Capacitor_SMD:C_0603_1608Metric_Pad1.08x0.95mm_HandSolder
- D2, D3, D4, D5: value D -> 1N4148; footprint Diode_THT:D_A-405_P7.62mm_Horizontal -> Diode_SMD:D_SOD-323_HandSoldering
- J1: value 908140508 -> FPC_Connector; footprint molex-picoflex8:CONN_SDA-90814_08_MOL -> Connector_FFC-FPC:JUSHUO_AFA07-S08FCA-00_1x8-1MP_P1.0mm_Horizontal
- R32: value 10k -> 1M
- R40, R41: value 100k -> 10k
- R6, R8: value 100k -> 1M
- RV1, RV2, RV3: value A10k -> A500k
- moved kibuzzard-67A4EC3B 87.2 mm to (171.8, 87.6)
- moved C23 71.8 mm to (64.1, 93.6), turned to 90 degrees
- moved C19 61.9 mm to (82.8, 80.9)
- moved kibuzzard-67A4EC49 60.7 mm to (175.1, 78.6)
- moved C9 47.8 mm to (120.5, 82.3), turned to 0 degrees
- moved C24 41.3 mm to (82.8, 109.7)
- moved C13 40.4 mm to (72.5, 93.6), turned to 90 degrees
- moved R23 40.1 mm to (113.4, 76.8)
- moved R20 34.9 mm to (110.1, 76.8), turned to -90 degrees
- moved R6 29.7 mm to (88.8, 109.7)
- moved C12 28.4 mm to (64.1, 103.9), turned to -90 degrees
- moved C21 27.0 mm to (108.8, 89.8)
- moved R22 20.5 mm to (128.7, 104.8), turned to -90 degrees
- moved D2 20.3 mm to (132.3, 116.6)
- moved R32 17.9 mm to (106.3, 89.8)
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Connections:
- C12 pad 2: /Core/Sum -> /Core/RetBuf
- C13 pad 2: /Core/PreFeedback -> /Core/OutPreVol
- C18 pad 1: Net-(C18-Pad1) -> /Core/InBuf
- C18 pad 2: /Snd -> Net-(C18-Pad2)
- C19 pad 1: Net-(C19-Pad1) -> /Core/FxOut
- C19 pad 2: /Out -> Net-(C19-Pad2)
- C21 pad 1: /+9V -> /GND
- C21 pad 2: /GND -> Net-(D9-K)
- C23 pad 2: Net-(C23-Pad2) -> /Core/InGain
- C24 pad 2: Net-(C24-Pad2) -> /Core/Feedback
- C7 pad 1: Net-(C7-Pad1) -> Net-(U1C-+)
- C7 pad 2: /Core/InBuf -> /GND
- C8 pad 1: Net-(C8-Pad1) -> Net-(U2B-+)
- C8 pad 2: /Core/RetBuf -> /GND
- C9 pad 2: /Core/OutPreVol -> Net-(C18-Pad2)
- D3 pad 2: /+4V5 -> /GND
- D5 pad 1: /+4V5 -> /GND
- R10 pad 2: Net-(C8-Pad1) -> Net-(C12-Pad1)
- R11 pad 2: Net-(C9-Pad1) -> Net-(C13-Pad1)
- R13 pad 1: /Core/InGain -> Net-(C23-Pad1)
- R14 pad 1: /Core/Feedback -> Net-(C24-Pad1)
- R18 pad 2: Net-(C12-Pad1) -> Net-(C32-Pad1)
- R19 pad 2: Net-(C13-Pad1) -> Net-(C33-Pad1)
- R22 pad 2: Net-(C23-Pad1) -> /Switching/JFET Switch 1/Out
- R23 pad 2: Net-(C24-Pad1) -> /Switching/JFET Switch 2/Out
- R26 pad 2: Net-(C18-Pad1) -> Net-(C36-Pad1)
- R27 pad 2: Net-(C19-Pad1) -> Net-(C37-Pad1)
- R32 pad 2: Net-(R32-Pad2) -> Net-(D9-K)
- R40 pad 2: Net-(C23-Pad2) -> Net-(U1B-+)
- R41 pad 2: Net-(C24-Pad2) -> Net-(U1A-+)
- R9 pad 2: Net-(C7-Pad1) -> Net-(C9-Pad1)
- RV1 pad 1: /+4V5 -> /GND
- RV1 pad 3: /Core/InBuf -> Net-(C18-Pad2)
- RV2 pad 1: /+4V5 -> /GND
- RV2 pad 2: /Core/FxOut -> Net-(C19-Pad2)
- RV3 pad 1: /+4V5 -> /GND
- U1 pad 10: Net-(C5-Pad2) -> Net-(U1C-+)
- U1 pad 3: Net-(C24-Pad2) -> Net-(U1A-+)
- U1 pad 5: Net-(C23-Pad2) -> Net-(U1B-+)
- U2 pad 5: Net-(C6-Pad2) -> Net-(U2B-+)
- U5 pad 3: Net-(R32-Pad2) -> /Switching/BypassState
- U5 pad 4: unconnected-(U5-Pad4) -> /Switching/~{BypassState}
- U5 pad 5: /GND -> /Switching/BypassState
- U5 pad 6: /GND -> /+9V
Routing:
- net /Core/FxOut: track 113.3 -> 0.00 mm, vias 2 -> 0
- net Net-(C32-Pad1): track 0.00 -> 85.8 mm, vias 0 -> 4
- net /Switching/BypassState: track 51.0 -> 0.00 mm, vias 2 -> 0
- net /Core/InBuf: track 47.5 -> 0.00 mm, vias 1 -> 0
- net Net-(C24-Pad2): track 47.1 -> 0.00 mm, vias 2 -> 0
- net /Snd: track 40.5 -> 0.00 mm
- net Net-(R32-Pad2): track 39.4 -> 0.00 mm, vias 2 -> 0
- net /+9V: track 244.9 -> 205.6 mm
- net Net-(C19-Pad1): track 37.7 -> 0.00 mm, vias 2 -> 0
- net /Core/Feedback: track 33.5 -> 0.00 mm
- net /Ret: track 36.4 -> 3.06 mm
- net /Core/RetBuf: track 78.6 -> 48.7 mm, vias 3 -> 2
- net /GND: track 111.6 -> 82.8 mm, vias 77 -> 59
- net Net-(C18-Pad1): track 24.9 -> 0.00 mm, vias 2 -> 0
- net Net-(SW1-B): track 53.5 -> 28.7 mm
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- removed copper zone on B.Cu, net /+4V5
- removed copper zone on F.Cu, net /+4V5
Other:
- board text removed: "JLCJLCJLCJLC"
