File: feedback-main-board/switching.kicad_sch (KiCad schematic)
At the start: 39 parts, among them Q2 MMBT3904, Q3 MMBT3904, Q4 MMBT3904, U1 TL074, U3 DG403, U4 NE555P, U5 4070

Commit message: Updates for rev2 schematic
Parts:
- removed C22: 100n, Capacitor_SMD:C_0603_1608Metric_Pad1.08x0.95mm_HandSolder, symbol Device:C
- removed U3: DG403, Package_SO:SOIC-16_3.9x9.9mm_P1.27mm, symbol pedals:DG403 Fixed
- removed U5: 4070, Package_SO:SOIC-14_3.9x8.7mm_P1.27mm, symbol 4xxx:4070
- added Q5: MMBT3904, Package_TO_SOT_SMD:SOT-23, symbol Transistor_BJT:MMBT3904
- added R31: 10k, Resistor_SMD:R_0603_1608Metric_Pad0.98x0.95mm_HandSolder, symbol Device:R
- added R42: 100k, Resistor_SMD:R_0603_1608Metric_Pad0.98x0.95mm_HandSolder, symbol Device:R
- added R43: 100, Resistor_SMD:R_0603_1608Metric_Pad0.98x0.95mm_HandSolder, symbol Device:R
- added U3: TMUX4053, Package_SO:TSSOP-16_4.4x5mm_P0.65mm, symbol pedals:TMUX4053
- C23, C24: value 100n -> 1u; footprint Capacitor_THT:C_Rect_L7.0mm_W2.5mm_P5.00mm -> Capacitor_THT:C_Rect_L7.0mm_W4.5mm_P5.00mm
- R22, R23: value 10k -> 100k
- U4: value NE555P -> NE555; Mouser 595-NE555PS -> 595-NE555DR
Connections:
- net +9V: now also R32.2, R31.1, U3.16 (V+)
- net BypassState: now also R42.2, U3.10 (SEL2), U3.11 (SEL1), U3.4 (D3); no longer R32.1
- net FxOut: now also U3.1 (S2B)
- net GND: now also Q5.2 (E), R42.1, R43.1, U3.7 (V-), U3.8 (Vref)
- net In: now also U3.12 (S1A)
- net LatchState: now also R30.1, U3.5 (S3A); no longer R30.2
- net RetBuf: now also U3.2 (S2A)
- net SignalSum: now also U3.13 (S1B)
- net at C23.1, R22.2: now also U3.14 (D1)
- net at C24.1, R23.2: now also U3.15 (D2)
- net MomSwIn renamed MomSw2
- net MomSw2: now also U3.9 (SEL3)
- new net: Q5.1 (B), R30.2
- new net: R43.2, U3.6 (~{EN})
- new net MomSw1: R31.2
- new net ~{LatchState}: Q5.3 (C), R32.1, U3.3 (S3B)
- no-connect marks 5 -> 2
Other:
- moved on the sheet: C18, C19, C21, C23, C24, R22, R23, R26, R27, R28, R29, R40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

Commit message: rev2 main board layout getting close
Parts:
- removed R43: 100, Resistor_SMD:R_0603_1608Metric_Pad0.98x0.95mm_HandSolder, symbol Device:R
Connections:
- net GND: now also U3.6 (~{EN})
Changed lines of the file:
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@@
-    (stroke (width 0) (type default) (color 0 0 0 0))
-  )
-  (wire (pts (xy 271.78 107.95) (xy 271.78 110.49))
     (stroke (width 0) (type default) (color 0 0 0 0))
   )
@@
     (stroke (width 0) (type default) (color 0 0 0 0))
   )
-  (wire (pts (xy 271.78 97.155) (xy 271.78 100.33))
+  (wire (pts (xy 271.78 97.155) (xy 271.78 110.49))
     (stroke (width 0) (type default) (color 0 0 0 0))
   )
@@
       (effects (font (size 1.27 1.27)) hide)
     )
-    (pin "1")
-    (pin "2")
-  )
-  (symbol (lib_id "Device:R") (at 271.78 104.14 180) (unit 1)
-    (in_bom yes) (on_board yes) (fields_autoplaced)
-    (property "Reference" "R43" (id 0) (at 273.685 102.8699 0)
-      (effects (font (size 1.27 1.27)) (justify right))
-    )
-    (property "Value" "100" (id 1) (at 273.685 105.4099 0)
-      (effects (font (size 1.27 1.27)) (justify right))
-    )
-    (property "Footprint" "Resistor_SMD:R_0603_1608Metric_Pad0.98x0.95mm_HandSolder" (id 2) (at 273.558 104.14 90)
-      (effects (font (size 1.27 1.27)) hide)
-    )
-    (property "Datasheet" "~" (id 3) (at 271.78 104.14 0)
-      (effects (font (size 1.27 1.27)) hide)
-    )
