File: feedback-main-board/switching.kicad_sch (KiCad schematic)
At the start: 39 parts, among them Q2 MMBT3904, Q3 MMBT3904, Q4 MMBT3904, U1 TL074, U3 DG403, U4 NE555, U5 CD4070

Commit message: JLCPCB rev3 ordered
Parts:
- C23, C24: value 100n -> 1u
- U1: value TL074 -> OPA1679; LCSC C6964 -> C2878631; Mouser 595-TL074IDR -> (none)
Changed lines of the file:
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@@
     (in_bom yes) (on_board yes) (fields_autoplaced)
     (property "Reference" "C23" (id 0) (at 90.805 35.56 90))
-    (property "Value" "100n" (id 1) (at 90.805 38.1 90))
+    (property "Value" "1u" (id 1) (at 90.805 38.1 90))
     (property "Footprint" "Capacitor_THT:C_Rect_L7.0mm_W2.5mm_P5.00mm" (id 2) (at 94.615 42.2148 0)
       (effects (font (size 1.27 1.27)) hide)
@@
     (in_bom yes) (on_board yes) (fields_autoplaced)
     (property "Reference" "C24" (id 0) (at 90.805 88.9 90))
-    (property "Value" "100n" (id 1) (at 90.805 91.44 90))
+    (property "Value" "1u" (id 1) (at 90.805 91.44 90))
     (property "Footprint" "Capacitor_THT:C_Rect_L7.0mm_W2.5mm_P5.00mm" (id 2) (at 94.615 95.5548 0)
       (effects (font (size 1.27 1.27)) hide)
@@
     (in_bom yes) (on_board yes) (fields_autoplaced)
     (property "Reference" "U1" (id 0) (at 103.505 83.82 0))
-    (property "Value" "TL074" (id 1) (at 103.505 86.36 0))
+    (property "Value" "OPA1679" (id 1) (at 103.505 86.36 0))
     (property "Footprint" "Package_SO:SOIC-14_3.9x8.7mm_P1.27mm" (id 2) (at 102.235 96.52 0)
       (effects (font (size 1.27 1.27)) hide)
@@
       (effects (font (size 1.27 1.27)) hide)
     )
-    (property "Mouser" "595-TL074IDR" (id 4) (at 103.505 93.98 0)
-      (effects (font (size 1.27 1.27)) hide)
-    )
-    (property "LCSC" "C6964" (id 5) (at 103.505 93.98 0)
+    (property "Mouser" "" (id 4) (at 103.505 93.98 0)
+      (effects (font (size 1.27 1.27)) hide)
+    )
+    (property "LCSC" "C2878631" (id 5) (at 103.505 93.98 0)
       (effects (font (size 1.27 1.27)) hide)
     )
@@
     (in_bom yes) (on_board yes) (fields_autoplaced)
     (property "Reference" "U1" (id 0) (at 103.505 30.48 0))
-    (property "Value" "TL074" (id 1) (at 103.505 33.02 0))
+    (property "Value" "OPA1679" (id 1) (at 103.505 33.02 0))
     (property "Footprint" "Package_SO:SOIC-14_3.9x8.7mm_P1.27mm" (id 2) (at 102.235 43.18 0)
       (effects (font (size 1.27 1.27)) hide)
@@
       (effects (font (size 1.27 1.27)) hide)
     )
-    (property "Mouser" "595-TL074IDR" (id 4) (at 103.505 40.64 0)
-      (effects (font (size 1.27 1.27)) hide)
-    )
-    (property "LCSC" "C6964" (id 5) (at 103.505 40.64 0)
-      (effects (font (size 1.27 1.27)) hide)
-    )
+    (property "Mouser" "" (id 4) (at 103.505 40.64 0)
+      (effects (font (size 1.27 1.27)) hide)
+    )
+    (property "LCSC" "C2878631" (id 5) (at 103.505 40.64 0)
+      (effects (font (size 1.27 1.27)) hide)
+    )
