File: feedback-main-board/switching.kicad_sch (KiCad schematic)
At the start: 39 parts, among them Q2 MMBT3904, Q3 MMBT3904, Q4 MMBT3904, U1 OPA1679, U3 DG403, U4 NE555, U5 CD4070

Commit message: wip
Parts:
- removed C21: 100n, Capacitor_SMD:C_0603_1608Metric_Pad1.08x0.95mm_HandSolder, symbol Device:C
- removed C23: 1u, Capacitor_THT:C_Rect_L7.0mm_W2.5mm_P5.00mm, symbol Device:C
- removed R32: 10k, Resistor_SMD:R_0603_1608Metric_Pad0.98x0.95mm_HandSolder, symbol Device:R
- removed U3: DG403, Package_SO:SOIC-16_3.9x9.9mm_P1.27mm, symbol pedals:DG403 Fixed
- added C?: 47u, Capacitor_SMD:CP_Elec_5x5.4, symbol Device:C_Polarized
- added TP1: BypassOff, TestPoint:TestPoint_Pad_D1.5mm, symbol Connector:TestPoint
- added TP2: BypassOn, TestPoint:TestPoint_Pad_D1.5mm, symbol Connector:TestPoint
- D6, D7, D8: now not fitted
- R40: value 100k -> 10k; LCSC C25803 -> C25804
Connections:
- net +9V: now also U5.6
- net BypassState: now also U5.3, U5.5, TP2.1
- net JFET Switch 1/Out: now reaches R22.2
- net JFET Switch 1/Out: now also C?.1
- net at R40.2, U1.5 (+): now also C?.2
- net JFET Switch 2/Out: now reaches C24.1, R23.2
- net ~{BypassState}: now reaches U5.4
- net ~{BypassState}: now also TP1.1
- net GND renamed SIG_GND
- net SIG_GND: no longer C17.2, C22.1, Q2.2 (E), Q3.2 (E), Q4.2 (E), U4.1 (GND), U5.5, U5.6, U5.7 (VSS)
- new net PWR_GND: C17.2, C22.1, Q2.2 (E), Q3.2 (E), Q4.2 (E), U4.1 (GND), U5.7 (VSS)
- no-connect marks 5 -> 4
Other:
- added sheet JFET Switch 1 (jfet-switch.kicad_sch)
- added sheet JFET Switch 2 (jfet-switch.kicad_sch)
- moved on the sheet: C16, C17, C20, C22, Q2, Q4, R21, R22, R24, R25, R29, R30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

Commit message: wip
Parts:
- removed C18, C19: 2u2, Capacitor_THT:C_Rect_L7.2mm_W7.2mm_P5.00mm_FKS2_FKP2_MKS2_MKP2, symbol Device:C
- removed C24: 1u, Capacitor_THT:C_Rect_L7.0mm_W2.5mm_P5.00mm, symbol Device:C
- added C35, C36, C37: 47u, Capacitor_SMD:CP_Elec_5x5.4, symbol Device:C_Polarized
- TP1, TP2: now not fitted; now left out of the parts list
- gave numbers to parts that had none: 1
Connections:
- net SIG_GND is gone; now on net GND: C16.1, C20.2, R25.2, R28.1, R29.1, R39.2, U5.12, U5.13, U5.8, U5.9
- net JFET Switch 2/Out: now also C35.1
- net Out: now also C37.2
- net Snd: now also C36.2
- net at R27.2: now also C37.1
- net at R41.2, U1.3 (+): now also C35.2
- net at R26.2: now also C36.1
- net PWR_GND renamed GND
Other:
- moved on the sheet: R23, R41, U1A

Commit message: wip pre grouping jfets
Parts:
- R41: value 100k -> 10k; LCSC C25803 -> C25804
Changed lines of the file:
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@@
 			)
 		)
-		(property "Value" "100k"
+		(property "Value" "10k"
 			(at 97.155 110.4899 0)
 			(show_name no)
@@
 			)
 		)
-		(property "LCSC" "C25803"
+		(property "LCSC" "C25804"
 			(at 95.25 109.22 0)
 			(hide yes)

Commit message: wip jacks board
Other:
- company: Pedal Markt / Andrei Salomatin -> Andrei Salomatin / akkusativ
- title: Read/Repeat -> RDRPT
- moved on the sheet: C16, C17, C22, R21, R24, R26, R27, R28, R30, R34, U1B, U4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
