File: feedback-main-board/jfet-switch.kicad_sch (KiCad schematic)
At the start: 11 parts, among them Q5 MMBFJ201, Q6 MMBFJ201

Commit message: wip
Parts:
- D10, D9: footprint Diode_SMD:D_SOD-323 -> Diode_SMD:D_SOD-323_HandSoldering
- TP3: now not fitted; now left out of the parts list
Changed lines of the file:
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@@
 			)
 		)
-		(property "Footprint" "Diode_SMD:D_SOD-323"
+		(property "Footprint" "Diode_SMD:D_SOD-323_HandSoldering"
 			(at 111.125 71.12 0)
 			(hide yes)
@@
 		(body_style 1)
 		(exclude_from_sim no)
-		(in_bom yes)
+		(in_bom no)
 		(on_board yes)
 		(in_pos_files yes)
-		(dnp no)
+		(dnp yes)
 		(fields_autoplaced yes)
 		(property "Reference" "TP3"
@@
 			)
 		)
-		(property "Footprint" "Diode_SMD:D_SOD-323"
+		(property "Footprint" "Diode_SMD:D_SOD-323_HandSoldering"
 			(at 201.295 71.12 0)
 			(hide yes)

Commit message: wip jacks board
Other:
- company: Pedal Markt / Andrei Salomatin -> Andrei Salomatin / akkusativ
- title: Read/Repeat -> RDRPT
Changed lines of the file:
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@@
 	(paper "A4")
 	(title_block
-		(title "Read/Repeat")
-		(date "2025-05-19")
-		(rev "v1rev4")
-		(company "Pedal Markt / Andrei Salomatin")
+		(title "RDRPT")
+		(date "2026-10-18")
+		(rev "v2rev1")
+		(company "Andrei Salomatin / akkusativ")
 	)
 	(junction
